File: mcu.kicad_sch (KiCad schematic)
At the start: 46 parts, among them J10 SWD, Cortex-M 10-pin 1.27 mm, Q20 2N7002, SW1 RESET (RUN to GND), SW2 BOOTSEL (via R24), U20 RP2354B, Y1 12 MHz ABM8-272-T3, CL 10 pF

Commit message: Physical design: VBAT-in buck, ESC pad row, pad-row IO, 50 mm single-sided board
Power: the FC now takes raw 2-6S VBAT from the MicoAir AM32 4-in-1 ESC pad
row (CURR TX M4 M3 M2 M1 VBAT GND, J3) through an AP63205WU 5 V/2 A buck
(U26, XGL4030-472, 3 x 22 uF) into the existing TPS2121 mux; XT30 and its
TVS removed. VBAT sense 100k/10k (36 V FS) on ADC0, ESC current sense on
ADC2, ESC KISS telemetry on GPIO30.

IO per the physical spec (DESIGN_SPEC "Physical design"): solder pad rows
for GPS/ELRS/MAG (JST-GH removed), DBG and buzzer; 3x4 servo block for
PWM5-8; 2x6 spare-IO block; WS2812C-2020 RGB LED replaces the two discrete
LEDs; buzzer moved off-board to pads; flash socket is the 150-mil SOIC-8
(W25Q64 default, APS6404L PSRAM alternative); four 4.0 mm grommet holes on
the 30.5 mm pattern. Passives moved to 0402/0603 for the single-sided
envelope.

Board: tools/setup_pcb.py regenerates MARV-V2.kicad_pcb from the netlist —
50 x 50 mm, 4-layer JLC 7628 stack-up, net classes incl. a 90 ohm USB pair,
edge-anchored connectors, coarse interior placement, silk pad labels.
DRC leaves only unrouted items. The BMP581 project footprint had its 2-pad
edges at +/-0.5 mm (corner pads overlapped, three nets shorted); corrected
to Bosch Fig. 32 (+/-0.25 mm, 0.20 mm gaps).

Checks: ERC 0/0, 217 pin mappings / 139 components, run_power_checks PASS,
audit 139/139, pcb DRC unrouted-only.

Co-Authored-By: Claude Fable 5.1 <noreply@anthropic.com>
Claude-Session: https://claude.ai/code/session_01U6Ud7JA3CDTJZVcZZr5sx1
Parts:
- removed BZ1: 5 V active buzzer, Buzzer_Beeper:Buzzer_12x9.5RM7.6, symbol Device:Buzzer
- removed D21: red, warning, LED_SMD:LED_0603_1608Metric, symbol Device:LED
- removed R31: 1k, green status LED, Resistor_SMD:R_0603_1608Metric, symbol Device:R
- removed R32: 1k, red warning LED, Resistor_SMD:R_0603_1608Metric, symbol Device:R
- added C78: 100n / 16 V X7R, ADC2 filter, Capacitor_SMD:C_0402_1005Metric, symbol Device:C
- added C79: 100n / 16 V X7R, D20 VDD, Capacitor_SMD:C_0402_1005Metric, symbol Device:C
- added H1, H2, H3, H4: M3 grommet hole, 4.0 mm NPTH, MARV_Packages:MountingHole_4.0mm_Grommet, symbol Mechanical:MountingHole
- added J15: BUZZER pads (5V BZ-), MARV_Packages:PadRow_1x02_P2.00mm, symbol Connector_Generic:Conn_01x02
- added J16: SPARE IO 2x6 (see note), Connector_PinHeader_2.54mm:PinHeader_2x06_P2.54mm_Vertical, symbol Connector_Generic:Conn_02x06_Odd_Even
- added R53: 1k / 1%, CURR series, Resistor_SMD:R_0402_1005Metric, symbol Device:R
- added R54: 1k, ESC telemetry series, Resistor_SMD:R_0402_1005Metric, symbol Device:R
- added R55: 100 / 1%, WS2812 data series, Resistor_SMD:R_0402_1005Metric, symbol Device:R
- C30, C31, C32, C33, C34, C35, C36, C37, C38, C40, C42, C43, C44, C48, C49: footprint Capacitor_SMD:C_0805_2012Metric -> Capacitor_SMD:C_0402_1005Metric
- C39: value 4.7u / 10 V X7R, VREG_VIN -> 4.7u / 10 V X7R 0603, VREG_VIN; footprint Capacitor_SMD:C_0805_2012Metric -> Capacitor_SMD:C_0603_1608Metric
- C41: value 4.7u / 10 V X7R, VREG_AVDD -> 4.7u / 10 V X7R 0603, VREG_AVDD; footprint Capacitor_SMD:C_0805_2012Metric -> Capacitor_SMD:C_0603_1608Metric
- C45: value 4.7u / 10 V X7R, DVDD bulk -> 4.7u / 10 V X7R 0603, DVDD bulk; footprint Capacitor_SMD:C_0805_2012Metric -> Capacitor_SMD:C_0603_1608Metric
- D20: value green, status -> WS2812C-2020 RGB; footprint LED_SMD:LED_0603_1608Metric -> MARV_Packages:LED_WS2812B-2020_PLCC4_2.0x2.0mm; symbol Device:LED -> LED:WS2812B-2020
- D22: value flyback across BZ1 -> flyback across the buzzer pads
- J10: value SWD, Cortex-M 10-pin 1.27 mm -> DBG pads (SWCLK SWDIO GND); footprint Connector_PinHeader_1.27mm:PinHeader_2x05_P1.27mm_Vertical_SMD -> MARV_Packages:PadRow_1x03_P2.00mm; symbol Connector_Generic:Conn_02x05_Odd_Even -> Connector_Generic:Conn_01x03
- R20, R21, R22, R23, R24, R25, R26, R29, R30, R33, R34: footprint Resistor_SMD:R_0603_1608Metric -> Resistor_SMD:R_0402_1005Metric
- R27: value 22k / 1%, 5V_IN top -> 100k / 1%, VBAT top; footprint Resistor_SMD:R_0603_1608Metric -> Resistor_SMD:R_0402_1005Metric
- R28: value 10k / 1%, 5V_IN bottom -> 10k / 1%, VBAT bottom; footprint Resistor_SMD:R_0603_1608Metric -> Resistor_SMD:R_0402_1005Metric
Connections:
- net LED1_A is gone; now on net GND: D20.2 (VSS)
- net BUZZ_D: now also J15.2 (Pin_2)
- net GND: now also C78.2, C79.2, J16.12 (Pin_12), J16.2 (Pin_2); no longer D20.1 (K), J10.5 (Pin_5), J10.9 (Pin_9)
- net PWR_GOOD: no longer J10.10 (Pin_10)
- net SWCLK: now also J10.1 (Pin_1); no longer J10.4 (Pin_4)
- net V3V3_SYS: now also J16.1 (Pin_1); no longer J10.1 (Pin_1)
- net V5_SYS: now also D20.4 (VDD), C79.1, J15.1 (Pin_1)
- net IO_GPIO21: now reaches U20.21 (GPIO21)
- net IO_GPIO21: now also J16.4 (Pin_4)
- net ESC_TELEM_RX: now reaches U20.38 (GPIO30)
- net ESC_TELEM_RX: now also R54.2
- net IO_GPIO31: now reaches U20.39 (GPIO31)
- net IO_GPIO31: now also J16.6 (Pin_6)
- net CURR_SENSE: now reaches U20.53 (GPIO42/ADC2)
- net CURR_SENSE: now also C78.1, R53.2
- net IO_GPIO43: now reaches U20.54 (GPIO43/ADC3)
- net IO_GPIO43: now also J16.7 (Pin_7)
- net IO_GPIO44: now reaches U20.55 (GPIO44/ADC4)
- net IO_GPIO44: now also J16.8 (Pin_8)
- net IO_GPIO45: now reaches U20.56 (GPIO45/ADC5)
- net IO_GPIO45: now also J16.9 (Pin_9)
- net IO_GPIO46: now reaches U20.57 (GPIO46/ADC6)
- net IO_GPIO46: now also J16.10 (Pin_10)
- net IO_GPIO47: now reaches U20.58 (GPIO47/ADC7)
- net IO_GPIO47: now also J16.11 (Pin_11)
- net IO_GPIO1: now reaches U20.78 (GPIO1)
- net IO_GPIO1: now also J16.3 (Pin_3)
- net 5V_IN renamed VBAT
- net LED_STAT renamed LED_DATA
- net LED_DATA: now also R55.1
- net LED_WARN renamed IO_GPIO27
- net IO_GPIO27: now also J16.5 (Pin_5)
- net VIN_SENSE renamed VBAT_SENSE
- new net CURR_SENSE_RAW: R53.1
- new net ESC_TELEM: R54.1
- new net LED_DIN: D20.3 (DIN), R55.2
- no-connect marks 13 -> 1
Other:
- note added: "GPIO MAP (pin = QFN-80 pin) GPIO0 77 FLASH_CS1 QMI CS1n, log flash select GPIO1 78 IO_GPIO1 spare -> J16 pin 3 GPIO2 79 PWM1 PWM1 A GPIO3 80 PWM2 PWM1 B GPIO4 1 PWM3 PWM2 A GPIO5 2 PWM4 PWM2 B GPIO6 3 MAG_SDA I2C1 SDA GPIO7 4 MAG_SCL I2C1 SCL GPIO8 6 ELRS_RX UART1 TX -> radio RX GPIO9 7 ELRS_TX UART1 RX <- radio TX GPIO10 8 PWM5 PWM5 A GPIO11 9 PWM6 PWM5 B GPIO12 11 GPS_RX UART0 TX -> GPS RX GPIO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"
- note added: "GPIO24 25 IMU_INT2 ICM-45686 INT2/FSYNC/CLKIN GPIO25 26 BARO_INT BMP581 INT GPIO26 27 LED_DATA WS2812C-2020 data, 100 R series (R55) GPIO27 28 IO_GPIO27 spare -> J16 pin 5 GPIO28 36 BUZZ_PWM buzzer gate drive GPIO29 37 HG_ACC_INT ADXL375 INT1 GPIO30 38 ESC_TELEM_RX ESC KISS telemetry in (PIO UART RX), 1k series R54 GPIO31 39 IO_GPIO31 spare -> J16 pin 6 GPIO32 40 SD_CLK microSD CLK (PIO) GPIO33 4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"
- note added: "J10 is a 3-pad SWD landing (SWCLK / SWDIO / GND), not a 10-pin Cortex header: the board carries solder pads for every bus (DESIGN_SPEC "Physical design"). The debugger reference 3V3 and the debugger-driven reset line of the old 2x05 header are both gone - power the board from VBAT or USB while debugging, and use SW1 (RUN via PWR_GOOD) for reset. RUN is still held by the TPS62913 power-good pull-u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"
- note added: "J16 SPARE IO (2.54 mm THT, right edge). 1 V3V3_SYS | 2 GND | 3 GPIO1 | 4 GPIO21 | 5 GPIO27 | 6 GPIO31 | 7 GPIO43* | 8 GPIO44* | 9 GPIO45* | 10 GPIO46* | 11 GPIO47* | 12 GND. * = ADC-capable (ADC3-ADC7); silk-mark those five at layout. These GPIOs are no longer no-connect, so every RP2354B GPIO now terminates somewhere: 39 on board functions and ports, 9 on this block."
- note added: "MECHANICAL: H1-H4 are the four 4.0 mm NPTH grommet holes on the standard 30.5 x 30.5 mm pattern, centred on the board, each with a 5.0 mm copper keepout and an 8.0 mm top-side courtyard for the grommet flange. No pins, no nets. See DESIGN_SPEC "Physical design"."
- note added: "TELEMETRY AND ANALOG INPUTS (100 nF at each ADC pin). VBAT_SENSE: R27/R28 100k/10k scale VBAT by 1/11, so the 3.3 V ADC full scale is 36.3 V. A 6S pack at its 25.2 V maximum reads 2.29 V and a 2S pack at 6.0 V reads 0.55 V, so the whole 2-6S window is on-scale with headroom; the divider draws 229 uA at 25.2 V. The old 5V_IN divider is gone with the 5 V input itself. CURR_SENSE: the ESC current-se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"
- note removed: "GPIO MAP (pin = QFN-80 pin) GPIO0 77 FLASH_CS1 QMI CS1n, log flash select GPIO1 78 (no connect) spare GPIO2 79 PWM1 PWM1 A GPIO3 80 PWM2 PWM1 B GPIO4 1 PWM3 PWM2 A GPIO5 2 PWM4 PWM2 B GPIO6 3 MAG_SDA I2C1 SDA GPIO7 4 MAG_SCL I2C1 SCL GPIO8 6 ELRS_RX UART1 TX -> radio RX GPIO9 7 ELRS_TX UART1 RX <- radio TX GPIO10 8 PWM5 PWM5 A GPIO11 9 PWM6 PWM5 B GPIO12 11 GPS_RX UART0 TX -> GPS RX GPIO13 12 GPS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"
- note removed: "GPIO24 25 IMU_INT2 ICM-45686 INT2/FSYNC/CLKIN GPIO25 26 BARO_INT BMP581 INT GPIO26 27 LED_STAT green status LED GPIO27 28 LED_WARN red warning LED GPIO28 36 BUZZ_PWM buzzer gate drive GPIO29 37 HG_ACC_INT ADXL375 INT1 GPIO30 38 (no connect) spare GPIO31 39 (no connect) spare GPIO32 40 SD_CLK microSD CLK (PIO) GPIO33 42 SD_CMD microSD CMD GPIO34 43 SD_D0 microSD DAT0 GPIO35 44 SD_D1 microSD DAT1 G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"
- note removed: "J10 pin 1 is 3V3 OUT for debugger reference only - never power the board from it. Pin 10 is the debugger reset line on PWR_GOOD/RUN; pins 6-8 (SWO, KEY, NC) unused. RUN is held by the TPS62913 power-good pull-up on POWER 2, so the MCU cannot run before V3V3_SYS is in regulation."
- note removed: "Telemetry dividers, 100 nF at each ADC pin. VIN_SENSE (R27/R28 22k/10k) scales by 10/32 = 0.3125, so the 3.3 V ADC full scale is 10.56 V: 1.56 V at 5.00 V in, 1.72 V at 5.50 V, and a 2S mis-plug at 8.4 V still reads on-scale (2.63 V) instead of pinning the input, which is the point of the wider divider. VBUS_SENSE keeps 10k/15k. Buzzer runs from V5_SYS (avionics OR output), never from the servo b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"
- moved on the sheet: C48, C49, D22, Q20, R27, R28, R29, R30, R33, R34

Commit message: Remove buzzer; passives to 0201/0402; GPIO28 to spare-IO block
Buzzer pads J15, driver Q20/D22/R33/R34 and the BUZZ nets removed; GPIO28
now terminates on J16 pin 12 (was a second GND). Resistors 0201, caps
<= 4.7 uF 0402, 22 uF/10 V 0603, 22 uF/25 V and 10 uF/50 V 0805, 47 uF
0805; USB net-class clearance 0.18 mm so the 0201 series resistors on the
pair pass DRC. Board regenerated at 50 x 50 mm (courtyard fill 63.5 %);
DRC unrouted-only. 134 components, 105 nets; ERC 0/0, 213 pin mappings,
run_power_checks PASS, audit 134/134.

Co-Authored-By: Claude Fable 5.1 <noreply@anthropic.com>
Claude-Session: https://claude.ai/code/session_01U6Ud7JA3CDTJZVcZZr5sx1
Parts:
- removed D22: flyback across the buzzer pads, Diode_SMD:D_SOD-123, symbol Device:D_Schottky
- removed J15: BUZZER pads (5V BZ-), MARV_Packages:PadRow_1x02_P2.00mm, symbol Connector_Generic:Conn_01x02
- removed Q20: 2N7002, Package_TO_SOT_SMD:SOT-23, symbol Transistor_FET:2N7002
- removed R33: 1k, gate series, Resistor_SMD:R_0402_1005Metric, symbol Device:R
- removed R34: 100k, gate pull-down, Resistor_SMD:R_0402_1005Metric, symbol Device:R
- C39: value 4.7u / 10 V X7R 0603, VREG_VIN -> 4.7u / 10 V X5R 0402, VREG_VIN; footprint Capacitor_SMD:C_0603_1608Metric -> Capacitor_SMD:C_0402_1005Metric
- C41: value 4.7u / 10 V X7R 0603, VREG_AVDD -> 4.7u / 10 V X5R 0402, VREG_AVDD; footprint Capacitor_SMD:C_0603_1608Metric -> Capacitor_SMD:C_0402_1005Metric
- C45: value 4.7u / 10 V X7R 0603, DVDD bulk -> 4.7u / 10 V X5R 0402, DVDD bulk; footprint Capacitor_SMD:C_0603_1608Metric -> Capacitor_SMD:C_0402_1005Metric
- R20, R21, R22, R23, R24, R25, R26, R27, R28, R29, R30, R53, R54, R55: footprint Resistor_SMD:R_0402_1005Metric -> Resistor_SMD:R_0201_0603Metric
Connections:
- net GND: no longer J16.12 (Pin_12)
- net BUZZ_PWM renamed IO_GPIO28
- net IO_GPIO28: now also J16.12 (Pin_12)
Other:
- note added: "GPIO24 25 IMU_INT2 ICM-45686 INT2/FSYNC/CLKIN GPIO25 26 BARO_INT BMP581 INT GPIO26 27 LED_DATA WS2812C-2020 data, 100 R series (R55) GPIO27 28 IO_GPIO27 spare -> J16 pin 5 GPIO28 36 IO_GPIO28 spare -> J16 pin 12 GPIO29 37 HG_ACC_INT ADXL375 INT1 GPIO30 38 ESC_TELEM_RX ESC KISS telemetry in (PIO UART RX), 1k series R54 GPIO31 39 IO_GPIO31 spare -> J16 pin 6 GPIO32 40 SD_CLK microSD CLK (PIO) GPIO3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"
- note added: "J16 SPARE IO (2.54 mm THT, right edge). 1 V3V3_SYS | 2 GND | 3 GPIO1 | 4 GPIO21 | 5 GPIO27 | 6 GPIO31 | 7 GPIO43* | 8 GPIO44* | 9 GPIO45* | 10 GPIO46* | 11 GPIO47* | 12 GPIO28. * = ADC-capable (ADC3-ADC7); silk-mark those five at layout. Pin 12 was the second ground; it now carries GPIO28, which the deleted buzzer driver used to own, so the block has one ground (pin 2) and ten GPIOs. These GPIOs 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"
- note removed: "GPIO24 25 IMU_INT2 ICM-45686 INT2/FSYNC/CLKIN GPIO25 26 BARO_INT BMP581 INT GPIO26 27 LED_DATA WS2812C-2020 data, 100 R series (R55) GPIO27 28 IO_GPIO27 spare -> J16 pin 5 GPIO28 36 BUZZ_PWM buzzer gate drive GPIO29 37 HG_ACC_INT ADXL375 INT1 GPIO30 38 ESC_TELEM_RX ESC KISS telemetry in (PIO UART RX), 1k series R54 GPIO31 39 IO_GPIO31 spare -> J16 pin 6 GPIO32 40 SD_CLK microSD CLK (PIO) GPIO33 4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"
- note removed: "J16 SPARE IO (2.54 mm THT, right edge). 1 V3V3_SYS | 2 GND | 3 GPIO1 | 4 GPIO21 | 5 GPIO27 | 6 GPIO31 | 7 GPIO43* | 8 GPIO44* | 9 GPIO45* | 10 GPIO46* | 11 GPIO47* | 12 GND. * = ADC-capable (ADC3-ADC7); silk-mark those five at layout. These GPIOs are no longer no-connect, so every RP2354B GPIO now terminates somewhere: 39 on board functions and ports, 9 on this block."

Commit message: IO array replaces bus pad rows; PINOUT.md pin plan; test points; ESC/battery docs
Left edge is now one 2 x 16 through-hole IO array (J6, signal | 5V/3V3/GND
rows, madflight-style) carrying GPS/ELRS/MAG and the ten spare GPIOs; the
J6/J7/J9 pad rows and the J16 block are gone. ESC pad row J3 and DBG pads
J10 stay; servo block J12-J14 stays beside the ESC row. TP1-TP10 1 mm test
points on the sensor SPI, chip selects and interrupts.

PINOUT.md records every GPIO's function and alternates from RP2350
datasheet Table 3, the spare-pin roles (I2C0 on 44/45, SPI1 on 46/47/28,
ADC3-7) and the peripheral ledger; check_power_netlist.py now asserts all
48 GPIO nets against it.

DESIGN_SPEC: ESC connection table, IO array table, test points, battery
monitoring (VBAT_SENSE + ESC current; INA226 rejected), edge allocation.
setup_pcb.py vendors the header footprints with project-local 3D models;
board 50 x 50 mm (48 collides with the grommet keepouts), DRC unrouted-only.
141 components, 105 nets, 231 pin mappings; ERC 0/0, ngspice PASS,
audit 141/141.

Co-Authored-By: Claude Fable 5.1 <noreply@anthropic.com>
Claude-Session: https://claude.ai/code/session_01U6Ud7JA3CDTJZVcZZr5sx1
Parts:
- removed J16: SPARE IO 2x6 (see note), Connector_PinHeader_2.54mm:PinHeader_2x06_P2.54mm_Vertical, symbol Connector_Generic:Conn_02x06_Odd_Even
Other:
- note added: "GPIO MAP (pin = QFN-80 pin) GPIO0 77 FLASH_CS1 QMI CS1n, log flash select GPIO1 78 IO_GPIO1 IO array -> J6 pin 23 GPIO2 79 PWM1 PWM1 A GPIO3 80 PWM2 PWM1 B GPIO4 1 PWM3 PWM2 A GPIO5 2 PWM4 PWM2 B GPIO6 3 MAG_SDA I2C1 SDA GPIO7 4 MAG_SCL I2C1 SCL GPIO8 6 ELRS_RX UART1 TX -> radio RX GPIO9 7 ELRS_TX UART1 RX <- radio TX GPIO10 8 PWM5 PWM5 A GPIO11 9 PWM6 PWM5 B GPIO12 11 GPS_RX UART0 TX -> GPS RX G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"
- note added: "GPIO24 25 IMU_INT2 ICM-45686 INT2/FSYNC/CLKIN GPIO25 26 BARO_INT BMP581 INT GPIO26 27 LED_DATA WS2812C-2020 data, 100 R series (R55) GPIO27 28 IO_GPIO27 IO array -> J6 pin 27 GPIO28 36 IO_GPIO28 IO array -> J6 pin 29 GPIO29 37 HG_ACC_INT ADXL375 INT1 GPIO30 38 ESC_TELEM_RX ESC KISS telemetry in (PIO UART RX), 1k series R54 GPIO31 39 IO_GPIO31 IO array -> J6 pin 31 GPIO32 40 SD_CLK microSD CLK (PI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"
- note added: "J10 is a 3-pad SWD landing (SWCLK / SWDIO / GND), not a 10-pin Cortex header: solder pads are kept for the two ports that mate with something fixed - the ESC row J3 and this one (DESIGN_SPEC "Connection philosophy"). The debugger reference 3V3 and the debugger-driven reset line of the old 2x05 header are both gone - power the board from VBAT or USB while debugging, and use SW1 (RUN via PWR_GOOD) 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"
- note added: "PORT NAMING: a port label is named for the peripheral pin it comes from, so GPS_TX / ELRS_TX are module outputs and land on MCU UART RX pins, while GPS_RX / ELRS_RX are module inputs fed by the MCU UART TX pins. On the J6 IO array (POWER 3) the UART rows are therefore 1 GPS_RX (silk T0) / 2 GPS_TX (R0) / 3 ELRS_RX (T1) / 4 ELRS_TX (R1), and rows 5/6 are MAG_SDA / MAG_SCL. The GPS and ELRS rows ta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"
- note added: "SPARE IO -> J6 (POWER 3, IO array 2x16, left edge). GPIO44 pin 13 | GPIO45 pin 15 | GPIO46 pin 17 | GPIO47 pin 19 | GPIO43 pin 21 | GPIO1 pin 23 | GPIO21 pin 25 | GPIO27 pin 27 | GPIO28 pin 29 | GPIO31 pin 31. GPIO43-47 are ADC3-ADC7; their silk labels are A43-A47 rather than IOnn to say so. Each of those odd pins has its own even neighbour: V3V3_SYS on odd rows, GND on even rows, so a spare GPIO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"
- note removed: "GPIO MAP (pin = QFN-80 pin) GPIO0 77 FLASH_CS1 QMI CS1n, log flash select GPIO1 78 IO_GPIO1 spare -> J16 pin 3 GPIO2 79 PWM1 PWM1 A GPIO3 80 PWM2 PWM1 B GPIO4 1 PWM3 PWM2 A GPIO5 2 PWM4 PWM2 B GPIO6 3 MAG_SDA I2C1 SDA GPIO7 4 MAG_SCL I2C1 SCL GPIO8 6 ELRS_RX UART1 TX -> radio RX GPIO9 7 ELRS_TX UART1 RX <- radio TX GPIO10 8 PWM5 PWM5 A GPIO11 9 PWM6 PWM5 B GPIO12 11 GPS_RX UART0 TX -> GPS RX GPIO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"
- note removed: "GPIO24 25 IMU_INT2 ICM-45686 INT2/FSYNC/CLKIN GPIO25 26 BARO_INT BMP581 INT GPIO26 27 LED_DATA WS2812C-2020 data, 100 R series (R55) GPIO27 28 IO_GPIO27 spare -> J16 pin 5 GPIO28 36 IO_GPIO28 spare -> J16 pin 12 GPIO29 37 HG_ACC_INT ADXL375 INT1 GPIO30 38 ESC_TELEM_RX ESC KISS telemetry in (PIO UART RX), 1k series R54 GPIO31 39 IO_GPIO31 spare -> J16 pin 6 GPIO32 40 SD_CLK microSD CLK (PIO) GPIO3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"
- note removed: "J10 is a 3-pad SWD landing (SWCLK / SWDIO / GND), not a 10-pin Cortex header: the board carries solder pads for every bus (DESIGN_SPEC "Physical design"). The debugger reference 3V3 and the debugger-driven reset line of the old 2x05 header are both gone - power the board from VBAT or USB while debugging, and use SW1 (RUN via PWR_GOOD) for reset. RUN is still held by the TPS62913 power-good pull-u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"
- note removed: "J16 SPARE IO (2.54 mm THT, right edge). 1 V3V3_SYS | 2 GND | 3 GPIO1 | 4 GPIO21 | 5 GPIO27 | 6 GPIO31 | 7 GPIO43* | 8 GPIO44* | 9 GPIO45* | 10 GPIO46* | 11 GPIO47* | 12 GPIO28. * = ADC-capable (ADC3-ADC7); silk-mark those five at layout. Pin 12 was the second ground; it now carries GPIO28, which the deleted buzzer driver used to own, so the block has one ground (pin 2) and ten GPIOs. These GPIOs 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"
- note removed: "PORT NAMING: a port label is named for the peripheral pin it comes from, so GPS_TX / ELRS_TX are module outputs and land on MCU UART RX pins, while GPS_RX / ELRS_RX are module inputs fed by the MCU UART TX pins. On J6/J7 (POWER 3, Pixhawk DS-009 order 1 VCC / 2 TX / 3 RX / 4 GND) pin 2 is therefore GPS_RX / ELRS_RX. J6 and J7 VCC are on V5_SYS; J9 VCC stays on V3V3_SYS. All port SIGNAL pins remai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"

Commit message: Madflight-style layout: 48.7 x 41.2 mm, ESC row left, 3x14 IO block right
Board re-laid out to the madflight FC3v2 arrangement and shrunk from the
50 x 50 square: rectangle 48.7 x 41.2 mm, 30.5 mm mounting square offset
(7.0 mm left margin for the vertical ESC pad row J3, 11.2 mm right margin
for the IO block), grommet keepout Ø6.5. The IO block is three abutting
1x14 rows J6/J7/J8 (signal | 5V/3V3 | GND per row): T0 R0 T1 R1 SDA SCL
S5-S8 A44-A47. The servo block and the 2x16 array are gone (actuators sheet
removed); GPIO 1/21/27/28/31/43 are no-connect (PINOUT.md, checker
updated). microSD ejects off the top edge, USB-C/RESET/BOOT/LED/DBG on the
bottom edge, sensors + test points between the MCU and the IO block.

Courtyard fill 75.7 %, 0 fit/geometry problems, DRC unrouted-only.
140 components; ERC 0/0, checker PASS, ngspice PASS, audit 140/140.
Known: the board-level silk labels on the ESC row and IO block are
mis-nudged by the label fixer (CURR/VBAT/A47 hidden) — silk pass pending.

Co-Authored-By: Claude Fable 5.1 <noreply@anthropic.com>
Claude-Session: https://claude.ai/code/session_01U6Ud7JA3CDTJZVcZZr5sx1
Connections:
- net IO_GPIO1: no longer names the net of U20.78 (GPIO1)
- net IO_GPIO21: no longer names the net of U20.21 (GPIO21)
- net IO_GPIO27: no longer names the net of U20.28 (GPIO27)
- net IO_GPIO28: no longer names the net of U20.36 (GPIO28)
- net IO_GPIO31: no longer names the net of U20.39 (GPIO31)
- net IO_GPIO43: no longer names the net of U20.54 (GPIO43/ADC3)
- no-connect marks 1 -> 7
Other:
- note added: "GPIO MAP (pin = QFN-80 pin) GPIO0 77 FLASH_CS1 QMI CS1n, log flash select GPIO1 78 (no connect) unexposed spare - no connect GPIO2 79 PWM1 PWM1 A GPIO3 80 PWM2 PWM1 B GPIO4 1 PWM3 PWM2 A GPIO5 2 PWM4 PWM2 B GPIO6 3 MAG_SDA I2C1 SDA GPIO7 4 MAG_SCL I2C1 SCL GPIO8 6 ELRS_RX UART1 TX -> radio RX GPIO9 7 ELRS_TX UART1 RX <- radio TX GPIO10 8 PWM5 PWM5 A -> J6 row 7 (S5) GPIO11 9 PWM6 PWM5 B -> J6 row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"
- note added: "GPIO24 25 IMU_INT2 ICM-45686 INT2/FSYNC/CLKIN GPIO25 26 BARO_INT BMP581 INT GPIO26 27 LED_DATA WS2812C-2020 data, 100 R series (R55) GPIO27 28 (no connect) unexposed spare - no connect GPIO28 36 (no connect) unexposed spare - no connect GPIO29 37 HG_ACC_INT ADXL375 INT1 GPIO30 38 ESC_TELEM_RX ESC KISS telemetry in (PIO UART RX), 1k series R54 GPIO31 39 (no connect) unexposed spare - no connect GP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"
- note added: "PORT NAMING: a port label is named for the peripheral pin it comes from, so GPS_TX / ELRS_TX are module outputs and land on MCU UART RX pins, while GPS_RX / ELRS_RX are module inputs fed by the MCU UART TX pins. On the IO array (POWER 3) the UART rows are therefore 1 GPS_RX (silk T0) / 2 GPS_TX (R0) / 3 ELRS_RX (T1) / 4 ELRS_TX (R1), rows 5/6 are MAG_SDA / MAG_SCL, rows 7-10 the PWM5-8 servo sign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"
- note added: "SPARE IO. EXPOSED (IO array J6 signal column, POWER 3): GPIO44 row 11 (A44) | GPIO45 row 12 (A45) | GPIO46 row 13 (A46) | GPIO47 row 14 (A47). All four are ADC4-ADC7, which is why the silk labels are A44-A47 rather than IOnn; each sits next to a V3V3_SYS pin (J7) and a GND pin (J8) in the same row. UNEXPOSED, NO-CONNECT: GPIO1, GPIO21, GPIO27, GPIO28, GPIO31, GPIO43 carry a no-connect flag on thi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"
- note removed: "GPIO MAP (pin = QFN-80 pin) GPIO0 77 FLASH_CS1 QMI CS1n, log flash select GPIO1 78 IO_GPIO1 IO array -> J6 pin 23 GPIO2 79 PWM1 PWM1 A GPIO3 80 PWM2 PWM1 B GPIO4 1 PWM3 PWM2 A GPIO5 2 PWM4 PWM2 B GPIO6 3 MAG_SDA I2C1 SDA GPIO7 4 MAG_SCL I2C1 SCL GPIO8 6 ELRS_RX UART1 TX -> radio RX GPIO9 7 ELRS_TX UART1 RX <- radio TX GPIO10 8 PWM5 PWM5 A GPIO11 9 PWM6 PWM5 B GPIO12 11 GPS_RX UART0 TX -> GPS RX G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"
- note removed: "GPIO24 25 IMU_INT2 ICM-45686 INT2/FSYNC/CLKIN GPIO25 26 BARO_INT BMP581 INT GPIO26 27 LED_DATA WS2812C-2020 data, 100 R series (R55) GPIO27 28 IO_GPIO27 IO array -> J6 pin 27 GPIO28 36 IO_GPIO28 IO array -> J6 pin 29 GPIO29 37 HG_ACC_INT ADXL375 INT1 GPIO30 38 ESC_TELEM_RX ESC KISS telemetry in (PIO UART RX), 1k series R54 GPIO31 39 IO_GPIO31 IO array -> J6 pin 31 GPIO32 40 SD_CLK microSD CLK (PI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"
- note removed: "PORT NAMING: a port label is named for the peripheral pin it comes from, so GPS_TX / ELRS_TX are module outputs and land on MCU UART RX pins, while GPS_RX / ELRS_RX are module inputs fed by the MCU UART TX pins. On the J6 IO array (POWER 3) the UART rows are therefore 1 GPS_RX (silk T0) / 2 GPS_TX (R0) / 3 ELRS_RX (T1) / 4 ELRS_TX (R1), and rows 5/6 are MAG_SDA / MAG_SCL. The GPS and ELRS rows ta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"
- note removed: "SPARE IO -> J6 (POWER 3, IO array 2x16, left edge). GPIO44 pin 13 | GPIO45 pin 15 | GPIO46 pin 17 | GPIO47 pin 19 | GPIO43 pin 21 | GPIO1 pin 23 | GPIO21 pin 25 | GPIO27 pin 27 | GPIO28 pin 29 | GPIO31 pin 31. GPIO43-47 are ADC3-ADC7; their silk labels are A43-A47 rather than IOnn to say so. Each of those odd pins has its own even neighbour: V3V3_SYS on odd rows, GND on even rows, so a spare GPIO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"
