File: mcu.kicad_sch (KiCad schematic)
At the start: 47 parts, among them J10 DBG pads (SWCLK SWDIO GND), SW1 RESET (RUN to GND), SW2 BOOTSEL (via R24), U20 RP2354B, Y1 12 MHz ABM8-272-T3, CL 10 pF

Commit message: JLCPCB sourcing: Basic-part refactor, LCSC numbers in the schematic, order files and audit
Parts audited line by line against JLCPCB's live catalogue (tools/jlc/,
reports/jlc-audit.md). Resistors move 0201 -> 0402 (JLC's Basic library has
no 0201 resistor), the U7 FB divider becomes 10k/3.16k 0.1 % (15.8k 0.1 % is
not stocked), Y1 becomes TAXM12M4RFBCCT2T (CL 12 pF) with 18 pF loads, L2/L3
become CJIANG FTC303020D2R2MBCA / FTC404030S4R7MGCA (stocked; Isat 5.5 A /
6.0 A at 30 %, footprints + models vendored from KiCad), the 22 uF/25 V and
10 uF lines move to Basic parts. The U24 default fit is W25Q32JVSNIQ (the
W25Q64JVSSIQ is a 208-mil part and never fitted the 150-mil socket).

Every fitted symbol carries a hidden LCSC property stamped from
tools/jlc/lcsc_map.csv; tools/jlc/export_jlc.py writes reports/jlc-bom.csv
and reports/jlc-cpl.csv (top-side SMT, headers unpopulated, U24 DNP).
Result: 46 unique parts, 16 Basic / 1 Preferred / 29 Extended (was 9/1/35),
extended-fee estimate $87 (was $105), $45.68 per board at 10 (was $52.97 with
L2 unsourced). DESIGN_SPEC gains a Manufacturing (JLCPCB) section with the
quote parameters. Board rebuilt (0 fit/geometry, DRC unrouted-only); ERC
0/0, checker PASS, ngspice PASS, audit 140/140.

Co-Authored-By: Claude Fable 5.1 <noreply@anthropic.com>
Claude-Session: https://claude.ai/code/session_01U6Ud7JA3CDTJZVcZZr5sx1
Parts:
- C30, C31, C32, C33, C34, C35, C36, C37, C38, C40, C42, C43, C44, C48, C49, C78, C79: LCSC (none) -> C1525
- C39, C41, C45: LCSC (none) -> C23733
- C46, C47: value 15p / 50 V C0G -> 18p / 50 V C0G; LCSC (none) -> C541431
- D20: LCSC (none) -> C2976072
- L20: LCSC (none) -> C48783272
- R20: footprint Resistor_SMD:R_0201_0603Metric -> Resistor_SMD:R_0402_1005Metric; LCSC (none) -> C25105
- R21, R24, R53, R54: footprint Resistor_SMD:R_0201_0603Metric -> Resistor_SMD:R_0402_1005Metric; LCSC (none) -> C11702
- R22, R23: footprint Resistor_SMD:R_0201_0603Metric -> Resistor_SMD:R_0402_1005Metric; LCSC (none) -> C2909343
- R25, R26: footprint Resistor_SMD:R_0201_0603Metric -> Resistor_SMD:R_0402_1005Metric; LCSC (none) -> C25900
- R27: footprint Resistor_SMD:R_0201_0603Metric -> Resistor_SMD:R_0402_1005Metric; LCSC (none) -> C25741
- R28, R29: footprint Resistor_SMD:R_0201_0603Metric -> Resistor_SMD:R_0402_1005Metric; LCSC (none) -> C25744
- R30: footprint Resistor_SMD:R_0201_0603Metric -> Resistor_SMD:R_0402_1005Metric; LCSC (none) -> C25756
- R55: footprint Resistor_SMD:R_0201_0603Metric -> Resistor_SMD:R_0402_1005Metric; LCSC (none) -> C25076
- SW1, SW2: LCSC (none) -> C231329
- U20: LCSC (none) -> C39843328
- Y1: value 12 MHz ABM8-272-T3, CL 10 pF -> 12 MHz TAXM12M4RFBCCT2T, CL 12 pF; LCSC (none) -> C133337
Other:
- note added: "Crystal circuit per design guide Sec 4. Y1 IS TAXM12M4RFBCCT2T (LCSC C133337), 12 MHz, SMD 3225 4-pad, CL = 12 pF - the ABM8-272-T3 the earlier revision named is not orderable at JLCPCB in any form (reports/jlc-audit.md section 1). LOAD CAPS FOLLOW THE CRYSTAL, NOT THE OTHER WAY ROUND: CL = C46*C47/(C46+C47) + Cstray, so C46/C47 are 18 pF C0G each (2 x 18 pF in series = 9 pF, plus ~3 pF of XIN/XT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"
- note removed: "Crystal circuit per design guide Sec 4: ABM8-272-T3, 15 pF each side (7.5 pF series + ~3 pF stray = 10.5 pF vs CL 10 pF), 1 k in the XOUT leg to limit drive with a 50 ohm ESR crystal. C38 is the single design-guide decoupling exception (pins 68+69 share it). VREG_AVDD RC = 33 ohm + 4.7 uF (design guide Sec 2.1), taken from V3V3_SYS; VREG_FB is tied to DVDD, VREG_PGND to GND, EP to GND."

Commit message: Schematic re-organised into 11 per-subsystem pages, drawn as wired blocks
Each subsystem now has its own sheet (RP2354B, USB/debug, ICM-45686, BMP581,
ADXL375, microSD, QSPI expansion, VBAT buck + ESC row, priority mux, 3.3 V
rail, IO block) with the IC's own decoupling, pull-ups, test points and
connectors placed beside it and wired, labels only for nets leaving the
block. Root sheet is an index. tools/build_power.py grows a small layout
engine (wire routing, junctions, decoupling ladders, note flow) with
self-checks for dangling wires and multi-net wire islands; the long design
notes are preserved verbatim as module constants.

Purely presentational: netlist fingerprint (tools/netlist_fingerprint.py,
new) is identical before and after, ERC 0, power checks pass. PCB footprint
paths re-pointed at the new sheet UUIDs by tools/relink_pcb_paths.py (new);
the board diff is path lines only, DRC unconnected count unchanged.
README/DESIGN_SPEC sheet lists updated; pre-change sheets and generator in
backups/pre-sheet-reorg-2026-09-16/.

Also carries the uncommitted work that preceded it: PCB routing, plane
stitching and route-analysis tools (tools/route_*.py, stitch_planes.py),
GPIO remap in PINOUT.md / check_power_netlist.py / setup_pcb.py, and the
grommet mounting-hole footprint update.

Co-Authored-By: Claude Fable 5.1 <noreply@anthropic.com>
Claude-Session: https://claude.ai/code/session_01Y51PayhRcgfdi3hVsfn4qg
Parts:
- removed C48: 100n / 16 V X7R, ADC0, Capacitor_SMD:C_0402_1005Metric, symbol Device:C
- removed C49: 100n / 16 V X7R, ADC1, Capacitor_SMD:C_0402_1005Metric, symbol Device:C
- removed C78: 100n / 16 V X7R, ADC2 filter, Capacitor_SMD:C_0402_1005Metric, symbol Device:C
- removed C79: 100n / 16 V X7R, D20 VDD, Capacitor_SMD:C_0402_1005Metric, symbol Device:C
- removed D20: WS2812C-2020 RGB, MARV_Packages:LED_WS2812B-2020_PLCC4_2.0x2.0mm, symbol LED:WS2812B-2020
- removed H1, H2, H3, H4: M3 grommet hole, 4.0 mm NPTH, MARV_Packages:MountingHole_4.0mm_Grommet, symbol Mechanical:MountingHole
- removed J10: DBG pads (SWCLK SWDIO GND), MARV_Packages:PadRow_1x03_P2.00mm, symbol Connector_Generic:Conn_01x03
- removed R22: 27 / 1%, USB D+ series, Resistor_SMD:R_0402_1005Metric, symbol Device:R
- removed R23: 27 / 1%, USB D- series, Resistor_SMD:R_0402_1005Metric, symbol Device:R
- removed R27: 100k / 1%, VBAT top, Resistor_SMD:R_0402_1005Metric, symbol Device:R
- removed R28: 10k / 1%, VBAT bottom, Resistor_SMD:R_0402_1005Metric, symbol Device:R
- removed R29: 10k / 1%, VBUS top, Resistor_SMD:R_0402_1005Metric, symbol Device:R
- removed R30: 15k / 1%, VBUS bottom, Resistor_SMD:R_0402_1005Metric, symbol Device:R
- removed R53: 1k / 1%, CURR series, Resistor_SMD:R_0402_1005Metric, symbol Device:R
- removed R54: 1k, ESC telemetry series, Resistor_SMD:R_0402_1005Metric, symbol Device:R
- removed R55: 100 / 1%, WS2812 data series, Resistor_SMD:R_0402_1005Metric, symbol Device:R
Connections:
- net BARO_CS: now also U20.13 (GPIO14); no longer U20.22 (GPIO22)
- net BARO_INT: now also U20.12 (GPIO13); no longer U20.26 (GPIO25)
- net ELRS_RX: now also U20.16 (GPIO16); no longer U20.6 (GPIO8)
- net ELRS_TX: now also U20.17 (GPIO17); no longer U20.7 (GPIO9)
- net ESC_TELEM_RX: now also U20.40 (GPIO32); no longer U20.38 (GPIO30)
- net GPS_RX: now also U20.25 (GPIO24); no longer U20.11 (GPIO12)
- net GPS_TX: now also U20.26 (GPIO25); no longer U20.12 (GPIO13)
- net HG_ACC_CS: now also U20.1 (GPIO4); no longer U20.17 (GPIO17)
- net HG_ACC_INT: now also U20.78 (GPIO1); no longer U20.37 (GPIO29)
- net IMU_CS: now also U20.4 (GPIO7); no longer U20.20 (GPIO20)
- net IMU_INT1: now also U20.3 (GPIO6); no longer U20.23 (GPIO23)
- net IMU_INT2: now also U20.79 (GPIO2); no longer U20.25 (GPIO24)
- net LED_DATA: now also U20.80 (GPIO3); no longer U20.27 (GPIO26)
- net MAG_SCL: now also U20.23 (GPIO23); no longer U20.4 (GPIO7)
- net MAG_SDA: now also U20.22 (GPIO22); no longer U20.3 (GPIO6)
- net PWM1: now also U20.54 (GPIO43/ADC3); no longer U20.79 (GPIO2)
- net PWM2: now also U20.48 (GPIO39); no longer U20.80 (GPIO3)
- net PWM3: now also U20.47 (GPIO38); no longer U20.1 (GPIO4)
- net PWM4: now also U20.45 (GPIO36); no longer U20.2 (GPIO5)
- net PWM5: now also U20.20 (GPIO20); no longer U20.8 (GPIO10)
- net PWM6: now also U20.19 (GPIO19); no longer U20.9 (GPIO11)
- net PWM7: now also U20.14 (GPIO15); no longer U20.13 (GPIO14)
- net PWM8: now also U20.2 (GPIO5); no longer U20.14 (GPIO15)
- net PWR_SRC_ST: now also U20.46 (GPIO37); no longer U20.48 (GPIO39)
- net SD_CLK: now also U20.42 (GPIO33); no longer U20.40 (GPIO32)
- net SD_CMD: now also U20.43 (GPIO34); no longer U20.42 (GPIO33)
- net SD_D0: now also U20.36 (GPIO28); no longer U20.43 (GPIO34)
- net SD_D1: now also U20.37 (GPIO29); no longer U20.44 (GPIO35)
- net SD_D2: now also U20.38 (GPIO30); no longer U20.45 (GPIO36)
- net SD_D3: now also U20.39 (GPIO31); no longer U20.46 (GPIO37)
- net SD_DET: now also U20.44 (GPIO35); no longer U20.47 (GPIO38)
- net SENS_MISO: now also U20.6 (GPIO8); no longer U20.16 (GPIO16)
- net SENS_MOSI: now also U20.9 (GPIO11); no longer U20.19 (GPIO19)
- net SENS_SCK: now also U20.8 (GPIO10); no longer U20.18 (GPIO18)
- net VBAT_SENSE: now also U20.52 (GPIO41/ADC1); no longer U20.49 (GPIO40/ADC0)
- net VBUS_SENSE: now also U20.49 (GPIO40/ADC0); no longer U20.52 (GPIO41/ADC1)
- no-connect marks 7 -> 6
Other:
- note added: "(pins 68+69 share it). VREG_AVDD RC = 33 ohm + 4.7 uF (design guide Sec 2.1), taken from V3V3_SYS; VREG_FB is tied to DVDD, VREG_PGND to GND, EP to GND."
- note added: "12 MHz crystal"
- note added: "BOARD 1 - RP2354B, QFN-80, 2 MB IN-PACKAGE QSPI FLASH. Digital rails on V3V3_SYS, core DVDD from the on-chip buck. Supply pins fan out on the left into one decoupling group per rail."
- note added: "GPIO MAP (pin = QFN-80 pin) GPIO0 77 FLASH_CS1 QMI CS1n, log flash select GPIO1 78 HG_ACC_INT ADXL375 INT1 GPIO2 79 IMU_INT2 ICM-45686 INT2/FSYNC/CLKIN GPIO3 80 LED_DATA WS2812C-2020 data, 100 R series (R55) GPIO4 1 HG_ACC_CS ADXL375 CS GPIO5 2 PWM8 PWM2 B -> J6 row 10 (S8) GPIO6 3 IMU_INT1 ICM-45686 INT1 GPIO7 4 IMU_CS ICM-45686 AP_CS GPIO8 6 SENS_MISO SPI1 RX GPIO9 7 (no connect) unexposed spar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"
- note added: "GPIO24 25 GPS_RX UART1 TX -> GPS RX GPIO25 26 GPS_TX UART1 RX <- GPS TX GPIO26 27 (no connect) unexposed spare - no connect GPIO27 28 (no connect) unexposed spare - no connect GPIO28 36 SD_D0 microSD DAT0 (PIO, GPIOBASE 16 window) GPIO29 37 SD_D1 microSD DAT1 (PIO, GPIOBASE 16 window) GPIO30 38 SD_D2 microSD DAT2 (PIO, GPIOBASE 16 window) GPIO31 39 SD_D3 microSD DAT3 (PIO, GPIOBASE 16 window) GPI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"
- note added: "I2C1 pull-ups"
- note added: "On-chip core regulator"
- note added: "Reset and BOOTSEL"
- note added: "SPARE IO. EXPOSED (IO array J6 signal column, POWER 3): GPIO44 row 11 (A44) | GPIO45 row 12 (A45) | GPIO46 row 13 (A46) | GPIO47 row 14 (A47). All four are ADC4-ADC7, which is why the silk labels are A44-A47 rather than IOnn; each sits next to a V3V3_SYS pin (J7) and a GND pin (J8) in the same row. UNEXPOSED, NO-CONNECT: GPIO9, GPIO12, GPIO18, GPIO21, GPIO26, GPIO27 carry a no-connect flag on thi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"
- note added: "Supply rails and decoupling"
- note removed: "GPIO MAP (pin = QFN-80 pin) GPIO0 77 FLASH_CS1 QMI CS1n, log flash select GPIO1 78 (no connect) unexposed spare - no connect GPIO2 79 PWM1 PWM1 A GPIO3 80 PWM2 PWM1 B GPIO4 1 PWM3 PWM2 A GPIO5 2 PWM4 PWM2 B GPIO6 3 MAG_SDA I2C1 SDA GPIO7 4 MAG_SCL I2C1 SCL GPIO8 6 ELRS_RX UART1 TX -> radio RX GPIO9 7 ELRS_TX UART1 RX <- radio TX GPIO10 8 PWM5 PWM5 A -> J6 row 7 (S5) GPIO11 9 PWM6 PWM5 B -> J6 row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"
- note removed: "GPIO24 25 IMU_INT2 ICM-45686 INT2/FSYNC/CLKIN GPIO25 26 BARO_INT BMP581 INT GPIO26 27 LED_DATA WS2812C-2020 data, 100 R series (R55) GPIO27 28 (no connect) unexposed spare - no connect GPIO28 36 (no connect) unexposed spare - no connect GPIO29 37 HG_ACC_INT ADXL375 INT1 GPIO30 38 ESC_TELEM_RX ESC KISS telemetry in (PIO UART RX), 1k series R54 GPIO31 39 (no connect) unexposed spare - no connect GP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"
- note removed: "J10 is a 3-pad SWD landing (SWCLK / SWDIO / GND), not a 10-pin Cortex header: solder pads are kept for the two ports that mate with something fixed - the ESC row J3 and this one (DESIGN_SPEC "Connection philosophy"). The debugger reference 3V3 and the debugger-driven reset line of the old 2x05 header are both gone - power the board from VBAT or USB while debugging, and use SW1 (RUN via PWR_GOOD) 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"
- note removed: "MECHANICAL: H1-H4 are the four 4.0 mm NPTH grommet holes on the standard 30.5 x 30.5 mm pattern, centred on the board, each with a 5.0 mm copper keepout and an 8.0 mm top-side courtyard for the grommet flange. No pins, no nets. See DESIGN_SPEC "Physical design"."
- note removed: "SPARE IO. EXPOSED (IO array J6 signal column, POWER 3): GPIO44 row 11 (A44) | GPIO45 row 12 (A45) | GPIO46 row 13 (A46) | GPIO47 row 14 (A47). All four are ADC4-ADC7, which is why the silk labels are A44-A47 rather than IOnn; each sits next to a V3V3_SYS pin (J7) and a GND pin (J8) in the same row. UNEXPOSED, NO-CONNECT: GPIO1, GPIO21, GPIO27, GPIO28, GPIO31, GPIO43 carry a no-connect flag on thi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"
- note removed: "TELEMETRY AND ANALOG INPUTS (100 nF at each ADC pin). VBAT_SENSE: R27/R28 100k/10k scale VBAT by 1/11, so the 3.3 V ADC full scale is 36.3 V. A 6S pack at its 25.2 V maximum reads 2.29 V and a 2S pack at 6.0 V reads 0.55 V, so the whole 2-6S window is on-scale with headroom; the divider draws 229 uA at 25.2 V. The old 5V_IN divider is gone with the 5 V input itself. CURR_SENSE: the ESC current-se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"
- moved on the sheet: C30, C31, C32, C33, C34, C35, C36, C37, C38, C39, C40, C41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
