File: mcu.kicad_sch (KiCad schematic)
At the start: 28 parts, among them SW1 RESET (RUN to GND), SW2 BOOTSEL (via R24), U20 RP2354B, Y1 12 MHz TAXM12M4RFBCCT2T, CL 1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

Commit message: Power tree: 5 V-in from an external BEC; drop pack buck, TPS2121 mux, TPS62913 stage and USB ESD
Reverses the "pack-powered from the ESC" decision, which was made without
the owner's agreement and inverted the stated requirement (5 V in from a
BEC between the ESC and the FC, so any 2-6S BEC or a 1S boost works
upstream). 140 -> 116 parts; JLC 46 -> 32 LCSC parts, 29 -> 17 Extended.

- J3 ESC row 1x08 -> 1x09: pad 7 5V_IN, pad 8 GND, pad 9 VBAT (sense only,
  feeds the R27/R28/C48 divider on GPIO41; no zone, dropped from Power class)
- USB/5V OR: Q1 AO3401A (gate on USB_VBUS, 100k pull-down) + D1 1N5819WS,
  both JLC Basic. IO-block 5 V rows, C19, C20, C21 move ahead of the FET
  onto 5V_IN; V5_SYS feeds only U7, U12 and the status LED
- 3.3 V system rail: AP63203WU-7 fixed 3.3 V buck on its datasheet
  application circuit (DS41326 Table 2; 4.7 uH FTC404030S reused per sec. 10)
  replaces TPS62913 + FB1 + 0.1 % divider + two-stage filter. JLC Basic has
  no synchronous buck at all, so this one Extended part is accepted
- U12 TPS7A2033 analog LDO kept; EN now tied to V3V3_SYS (PWR_GOOD gone)
- PWR_SRC_ST gone, GPIO37 freed (no-connect); R10 becomes the MCU_RUN pull-up
- U8 USBLC6 (Extended) removed; D+/D- straight to the 27 R series resistors
- ngspice decks that modelled the removed chain retired to
  simulations/superseded/; run_power_checks.py reports RETIRED, not PASS
- DESIGN_SPEC decisions, README, LIBRARIES, PINOUT, BOM, JLC files and
  reports regenerated

Also carries the pre-session working-tree changes (grommet footprint
MountingHole_4.0mm_Grommet -> _Pad_Via, setup_pcb floorplan, JLC tooling).

Verified: ERC 0 violations; check_power_netlist PASS (5V_IN/V5_SYS/VBAT
membership asserted); setup_pcb 0 fit/geometry problems; stitch 150 vias;
DRC 5 silk_edge_clearance warnings only (board unrouted by design);
audit_footprints 116/116; JLC live audit 0 unresolved fitted parts;
generators idempotent modulo UUIDs.

Co-Authored-By: Claude Fable 5.1 <noreply@anthrop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
Parts:
- added R10: 100k, RUN pull-up, Resistor_SMD:R_0402_1005Metric, symbol Device:R
Connections:
- net V3V3_SYS: now also R10.1
- net PWR_GOOD renamed MCU_RUN
- net MCU_RUN: now also R10.2
- net PWR_SRC_ST: no longer names the net of U20.46 (GPIO37)
- no-connect marks 6 -> 7
