File: mcu.kicad_sch (KiCad schematic)
At the start: 29 parts, among them SW1 RESET (RUN to GND), SW2 BOOTSEL (via R24), U20 RP2354B, Y1 12 MHz TAXM12M4RFBCCT2T, CL 1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

Commit message: updoot
Parts:
- added R58: 22, Resistor_SMD:R_0402_1005Metric, symbol Device:R
Connections:
- net LED_DATA: now also U20.42 (GPIO33); no longer U20.80 (GPIO3)
- net SD_CLK: now also R58.2; no longer U20.42 (GPIO33)
- net SD_CMD: now also U20.28 (GPIO27); no longer U20.43 (GPIO34)
- net BARO_SDA: now reaches U20.11 (GPIO12)
- net ICM_INT2: now reaches U20.18 (GPIO18)
- net ADXL_INT2: now reaches U20.21 (GPIO21)
- net SD_CLK_MCU: now reaches U20.27 (GPIO26)
- net SD_CLK_MCU: now also R58.1
- net BARO_SCL: now reaches U20.7 (GPIO9)
- net BARO_CS renamed ADXL_CS
- net HG_ACC_CS renamed ADXL_MISO
- net HG_ACC_INT renamed ADXL_INT1
- net IMU_CS renamed ICM_CS
- net IMU_INT1 renamed ICM_INT1
- net IMU_INT2 renamed ADXL_SCK
- net SD_D0 renamed SD_DAT0
- net SD_D1 renamed SD_DAT1
- net SD_D2 renamed SD_DAT2
- net SD_D3 renamed SD_DAT3
- net SENS_MISO renamed ICM_MISO
- net SENS_MOSI renamed ICM_MOSI
- net SENS_SCK renamed ICM_SCK
- new net ADXL_MOSI: U20.80 (GPIO3)
- no-connect marks 7 -> 2
Other:
- note added: "GPIO MAP (pin = QFN-80 pin) GPIO0 77 FLASH_CS1 QMI CS1n, log flash select GPIO1 78 ADXL_INT1 ADXL375 INT1 GPIO2 79 ADXL_SCK SPI0 SCK GPIO3 80 ADXL_MOSI SPI0 TX GPIO4 1 ADXL_MISO SPI0 RX GPIO5 2 PWM8 PWM2 B -> J6 row 10 (S8) GPIO6 3 ICM_INT1 ICM-45686 INT1 GPIO7 4 ICM_CS ICM-45686 CS GPIO8 6 ICM_MISO SPI1 RX GPIO9 7 BARO_SCL I2C0 SCL GPIO10 8 ICM_SCK SPI1 SCK GPIO11 9 ICM_MOSI SPI1 TX GPIO12 11 BA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"
- note added: "GPIO24 25 GPS_RX UART1 TX -> GPS RX GPIO25 26 GPS_TX UART1 RX <- GPS TX GPIO26 27 SD_CLK_MCU PIO native SD clock -> R58 22R -> SD_CLK GPIO27 28 SD_CMD PIO native SD command GPIO28 36 SD_DAT0 native SD DAT0 GPIO29 37 SD_DAT1 native SD DAT1 GPIO30 38 SD_DAT2 native SD DAT2 GPIO31 39 SD_DAT3 native SD DAT3 GPIO32 40 ESC_TELEM_RX ESC KISS telemetry in (PIO UART RX, window 16-47), 1k series R54 GPIO33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"
- note added: "SD source-series damping R58: place next to U20 GPIO26. 22 ohm nominal; tune 0-33 ohm. No pull resistor on SD_CLK."
- note added: "SPARE IO: GPIO44-47 remain on IO block J6 rows 11-14. GPIO34 and GPIO37 are unexposed and carry no-connect flags. GPIO budget: 42 assigned, 4 exposed spares, 2 unconnected. SPI0: ADXL375 only. SPI1: ICM-45686 only. I2C0: BMP581 only. Native SD: GPIO26-31, PIO + DMA. Independent sensor interrupts. See PINOUT.md for the complete allocation."
- note removed: "GPIO MAP (pin = QFN-80 pin) GPIO0 77 FLASH_CS1 QMI CS1n, log flash select GPIO1 78 HG_ACC_INT ADXL375 INT1 GPIO2 79 IMU_INT2 ICM-45686 INT2/FSYNC/CLKIN GPIO3 80 LED_DATA WS2812C-2020 data, 100 R series (R55) GPIO4 1 HG_ACC_CS ADXL375 CS GPIO5 2 PWM8 PWM2 B -> J6 row 10 (S8) GPIO6 3 IMU_INT1 ICM-45686 INT1 GPIO7 4 IMU_CS ICM-45686 AP_CS GPIO8 6 SENS_MISO SPI1 RX GPIO9 7 (no connect) unexposed spar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"
- note removed: "GPIO24 25 GPS_RX UART1 TX -> GPS RX GPIO25 26 GPS_TX UART1 RX <- GPS TX GPIO26 27 (no connect) unexposed spare - no connect GPIO27 28 (no connect) unexposed spare - no connect GPIO28 36 SD_D0 microSD DAT0 (PIO, GPIOBASE 16 window) GPIO29 37 SD_D1 microSD DAT1 (PIO, GPIOBASE 16 window) GPIO30 38 SD_D2 microSD DAT2 (PIO, GPIOBASE 16 window) GPIO31 39 SD_D3 microSD DAT3 (PIO, GPIOBASE 16 window) GPI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"
- note removed: "SPARE IO. EXPOSED (IO array J6 signal column, POWER 3): GPIO44 row 11 (A44) | GPIO45 row 12 (A45) | GPIO46 row 13 (A46) | GPIO47 row 14 (A47). All four are ADC4-ADC7, which is why the silk labels are A44-A47 rather than IOnn; each sits next to a V3V3_SYS pin (J7) and a GND pin (J8) in the same row. UNEXPOSED, NO-CONNECT: GPIO9, GPIO12, GPIO18, GPIO21, GPIO26, GPIO27 carry a no-connect flag on thi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"

Commit message: Save communication schematic, locking microSD and manual PCB updates
Connections:
- net SD_DET: no longer names the net of U20.44 (GPIO35)
- no-connect marks 2 -> 3
Other:
- note added: "SPARE IO: GPIO44-47 remain on IO block J6 rows 11-14. GPIO34, GPIO35 and GPIO37 are unexposed and carry no-connect flags. GPIO budget: 41 assigned, 4 exposed spares, 3 unconnected. SPI0: ADXL375 only. SPI1: ICM-45686 only. I2C0: BMP581 only. Native SD: GPIO26-31, PIO + DMA. Independent sensor interrupts. See PINOUT.md for the complete allocation."
- note removed: "SPARE IO: GPIO44-47 remain on IO block J6 rows 11-14. GPIO34 and GPIO37 are unexposed and carry no-connect flags. GPIO budget: 42 assigned, 4 exposed spares, 2 unconnected. SPI0: ADXL375 only. SPI1: ICM-45686 only. I2C0: BMP581 only. Native SD: GPIO26-31, PIO + DMA. Independent sensor interrupts. See PINOUT.md for the complete allocation."

Commit message: update
Connections:
- net CURR_SENSE: now also U20.52 (GPIO41/ADC1); no longer U20.53 (GPIO42/ADC2)
- net ESC_TELEM_RX: now also U20.43 (GPIO34); no longer U20.40 (GPIO32)
- net LED_DATA: now also U20.54 (GPIO43/ADC3); no longer U20.42 (GPIO33)
- net PWM1: now also U20.48 (GPIO39); no longer U20.54 (GPIO43/ADC3)
- net PWM2: now also U20.47 (GPIO38); no longer U20.48 (GPIO39)
- net PWM3: now also U20.46 (GPIO37); no longer U20.47 (GPIO38)
- net SD_CLK_MCU: now also U20.40 (GPIO32); no longer U20.27 (GPIO26)
- net SD_CMD: now also U20.42 (GPIO33); no longer U20.28 (GPIO27)
- net VBAT_SENSE: now also U20.53 (GPIO42/ADC2); no longer U20.52 (GPIO41/ADC1)
Other:
- note added: "GPIO24 25 GPS_RX UART1 TX -> GPS RX GPIO25 26 GPS_TX UART1 RX <- GPS TX GPIO26 27 (no connect) unexposed spare - no connect GPIO27 28 (no connect) unexposed spare - no connect GPIO28 36 SD_DAT0 native SD DAT0 GPIO29 37 SD_DAT1 native SD DAT1 GPIO30 38 SD_DAT2 native SD DAT2 GPIO31 39 SD_DAT3 native SD DAT3 GPIO32 40 SD_CLK_MCU PIO native SD clock -> R58 22R -> SD_CLK (window 16-47) GPIO33 42 SD_C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"
- note added: "SD source-series damping R58: place next to U20 GPIO32 (pin 40). 22 ohm nominal; tune 0-33 ohm. No pull resistor on SD_CLK."
- note added: "SPARE IO: GPIO44-47 remain on IO block J6 rows 11-14. GPIO26, GPIO27 and GPIO35 are unexposed and carry no-connect flags. GPIO budget: 41 assigned, 4 exposed spares, 3 unconnected. SPI0: ADXL375 only. SPI1: ICM-45686 only. I2C0: BMP581 only. Native SD: GPIO28-33, PIO + DMA (window 16-47). Independent sensor interrupts. See PINOUT.md for the complete allocation."
- note removed: "GPIO24 25 GPS_RX UART1 TX -> GPS RX GPIO25 26 GPS_TX UART1 RX <- GPS TX GPIO26 27 SD_CLK_MCU PIO native SD clock -> R58 22R -> SD_CLK GPIO27 28 SD_CMD PIO native SD command GPIO28 36 SD_DAT0 native SD DAT0 GPIO29 37 SD_DAT1 native SD DAT1 GPIO30 38 SD_DAT2 native SD DAT2 GPIO31 39 SD_DAT3 native SD DAT3 GPIO32 40 ESC_TELEM_RX ESC KISS telemetry in (PIO UART RX, window 16-47), 1k series R54 GPIO33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"
- note removed: "SD source-series damping R58: place next to U20 GPIO26. 22 ohm nominal; tune 0-33 ohm. No pull resistor on SD_CLK."
- note removed: "SPARE IO: GPIO44-47 remain on IO block J6 rows 11-14. GPIO34, GPIO35 and GPIO37 are unexposed and carry no-connect flags. GPIO budget: 41 assigned, 4 exposed spares, 3 unconnected. SPI0: ADXL375 only. SPI1: ICM-45686 only. I2C0: BMP581 only. Native SD: GPIO26-31, PIO + DMA. Independent sensor interrupts. See PINOUT.md for the complete allocation."
