File: mcu.kicad_sch (KiCad schematic)
At the start: 30 parts, among them SW1 RESET (RUN to GND), SW2 BOOTSEL (via R24), U20 RP2354B, Y1 12 MHz TAXM12M4RFBCCT2T, CL 1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

Commit message: Order-ready: U24 via cleared, R58 sourced (C25092), fab and assembly exports
- Owner moved the GND via out of U24's pad column: DRC now has no electrical
  errors, 0 unconnected, 0 schematic-parity issues (78 cosmetic courtyard
  gaps and 80 RP2350 pad-size review warnings remain).
- R58 22 ohm 0402 gets LCSC C25092 in the schematic, the footprint field and
  tools/jlc/lcsc_map.csv.
- build/ (ignored) holds Gerbers+drill (build/MARV-V2-gerbers.zip) and the
  JLC BOM/CPL (build/assembly/) generated from this commit.

Co-Authored-By: Claude Fable 5.1 <noreply@anthropic.com>
Claude-Session: https://claude.ai/code/session_01VST8gLViyNpcDEYyh3itUW
Parts:
- R58: LCSC (none) -> C25092
Changed lines of the file:
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@@
+			)
+		)
+		(property "LCSC" "C25092"
+			(at 347.98 189.23 0)
+			(hide yes)
+			(show_name no)
+			(do_not_autoplace no)
+			(effects
+				(font
+					(size 1 1)
+				)
+				(justify left)
 			)
 		)
