File: mcu.kicad_sch (KiCad schematic)
At the start: 30 parts, among them SW1 RESET (RUN to GND), SW2 BOOTSEL (via R24), U20 RP2354B, Y1 12 MHz TAXM12M4RFBCCT2T, CL 1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

Commit message: DRC 0 err
Parts:
- L20: value 3.3u, 0806 AOTA-B201610S3R3 -> 3.3u, 0806 AOTA-B201610S3R3-101-T; LCSC C48783272 -> C42411119
Changed lines of the file:
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@@
 			)
 		)
-		(property "Value" "3.3u, 0806 AOTA-B201610S3R3"
+		(property "Value" "3.3u, 0806 AOTA-B201610S3R3-101-T"
 			(at 296.33 44.45 270)
 			(show_name no)
@@
 			)
 		)
-		(property "LCSC" "C48783272"
+		(property "LCSC" "C42411119"
 			(at 307.34 55.88 270)
 			(hide yes)
