File: io_block.kicad_sch (KiCad schematic)
At the start: 13 parts, among them J6 IO array signal column (inner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, J7 IO array power column (5V / 3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, J8 IO array GND column (board ed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

Commit message: Power tree: 5 V-in from an external BEC; drop pack buck, TPS2121 mux, TPS62913 stage and USB ESD
Reverses the "pack-powered from the ESC" decision, which was made without
the owner's agreement and inverted the stated requirement (5 V in from a
BEC between the ESC and the FC, so any 2-6S BEC or a 1S boost works
upstream). 140 -> 116 parts; JLC 46 -> 32 LCSC parts, 29 -> 17 Extended.

- J3 ESC row 1x08 -> 1x09: pad 7 5V_IN, pad 8 GND, pad 9 VBAT (sense only,
  feeds the R27/R28/C48 divider on GPIO41; no zone, dropped from Power class)
- USB/5V OR: Q1 AO3401A (gate on USB_VBUS, 100k pull-down) + D1 1N5819WS,
  both JLC Basic. IO-block 5 V rows, C19, C20, C21 move ahead of the FET
  onto 5V_IN; V5_SYS feeds only U7, U12 and the status LED
- 3.3 V system rail: AP63203WU-7 fixed 3.3 V buck on its datasheet
  application circuit (DS41326 Table 2; 4.7 uH FTC404030S reused per sec. 10)
  replaces TPS62913 + FB1 + 0.1 % divider + two-stage filter. JLC Basic has
  no synchronous buck at all, so this one Extended part is accepted
- U12 TPS7A2033 analog LDO kept; EN now tied to V3V3_SYS (PWR_GOOD gone)
- PWR_SRC_ST gone, GPIO37 freed (no-connect); R10 becomes the MCU_RUN pull-up
- U8 USBLC6 (Extended) removed; D+/D- straight to the 27 R series resistors
- ngspice decks that modelled the removed chain retired to
  simulations/superseded/; run_power_checks.py reports RETIRED, not PASS
- DESIGN_SPEC decisions, README, LIBRARIES, PINOUT, BOM, JLC files and
  reports regenerated

Also carries the pre-session working-tree changes (grommet footprint
MountingHole_4.0mm_Grommet -> _Pad_Via, setup_pcb floorplan, JLC tooling).

Verified: ERC 0 violations; check_power_netlist PASS (5V_IN/V5_SYS/VBAT
membership asserted); setup_pcb 0 fit/geometry problems; stitch 150 vias;
DRC 5 silk_edge_clearance warnings only (board unrouted by design);
audit_footprints 116/116; JLC live audit 0 unresolved fitted parts;
generators idempotent modulo UUIDs.

Co-Authored-By: Claude Fable 5.1 <noreply@anthrop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
Parts:
- H1, H2, H3, H4: value M3 grommet hole, 4.0 mm NPTH -> M3 grommet hole, 4.0 mm, GND ring; footprint MARV_Packages:MountingHole_4.0mm_Grommet -> MARV_Packages:MountingHole_4.0mm_Grommet_Pad_Via; symbol Mechanical:MountingHole -> Mechanical:MountingHole_Pad
Connections:
- net GND: now also H1.1, H2.1, H3.1, H4.1
- net V5_SYS: no longer C20.1, C21.1, J7.1 (Pin_1), J7.10 (Pin_10), J7.2 (Pin_2), J7.3 (Pin_3), J7.4 (Pin_4), J7.7 (Pin_7), J7.8 (Pin_8), J7.9 (Pin_9)
- new net 5V_IN: C20.1, C21.1, J7.1 (Pin_1), J7.10 (Pin_10), J7.2 (Pin_2), J7.3 (Pin_3), J7.4 (Pin_4), J7.7 (Pin_7), J7.8 (Pin_8), J7.9 (Pin_9)
Other:
- note added: "C20 / C21: 5V_IN local bulk at the array (rows 1-4 GPS/ELRS and rows 7-10 servo, the 5 V supply rows). C22: V3V3_SYS local bulk at the array (rows 5-6 and 11-14)."
- note added: "IO ARRAY ROW MAP (row n = J6 pin n signal | J7 pin n power | J8 pin n GND) 1 T0 GPS_RX | 5V_IN | GND UART1 TX -> GPS RX (GPIO24) 2 R0 GPS_TX | 5V_IN | GND UART1 RX <- GPS TX (GPIO25) 3 T1 ELRS_RX | 5V_IN | GND UART0 TX -> ELRS RX (GPIO16) 4 R1 ELRS_TX | 5V_IN | GND UART0 RX <- ELRS TX (GPIO17) 5 SDA MAG_SDA | V3V3_SYS | GND I2C1 SDA (GPIO22), 4.7k pull-up on the MCU sheet 6 SCL MAG_SCL | V3V3_SYS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"
- note added: "MECHANICAL: H1-H4 are the four 4.0 mm grommet holes on the standard 30.5 x 30.5 mm pattern, off-centre in X, each now a PLATED hole with a 6.4 mm GND pad ring stitched by eight 0.6/0.3 mm vias, and a 6.5 mm top-side courtyard for the grommet flange. Pin 1 of every hole is GND, so the frame screws bond to the ground plane on every layer. See DESIGN_SPEC "Mounting and orientation"."
- note added: "PWM MAP PWM5 = GPIO20 (row 7, S5) PWM6 = GPIO19 (row 8, S6) PWM7 = GPIO15 (row 9, S7) PWM8 = GPIO5 (row 10, S8) ON THE ESC PAD ROW (J3, POWER 1) PWM1 = GPIO43"
- note added: "PWM2 = GPIO39 PWM3 = GPIO38 PWM4 = GPIO36"
- note added: "RAILS ON THE ARRAY: rows 1-4 (GPS, ELRS) and rows 7-10 (servos S5-S8) take 5V_IN; rows 5-6 (magnetometer) and rows 11-14 (the four exposed spares) take V3V3_SYS. Every row has its own GND pin in the J8 column, so a signal return is never more than 2.54 mm away and no row can be mis-plugged into a neighbour's ground. THE EIGHT 5 V ROWS ARE ON 5V_IN, AHEAD OF THE OR-ING FET (DESIGN_SPEC "Decisions"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"
- note removed: "C20 / C21: V5_SYS local bulk at the array (rows 1-4 GPS/ELRS and rows 7-10 servo, the 5 V supply rows). C22: V3V3_SYS local bulk at the array (rows 5-6 and 11-14)."
- note removed: "IO ARRAY ROW MAP (row n = J6 pin n signal | J7 pin n power | J8 pin n GND) 1 T0 GPS_RX | V5_SYS | GND UART1 TX -> GPS RX (GPIO24) 2 R0 GPS_TX | V5_SYS | GND UART1 RX <- GPS TX (GPIO25) 3 T1 ELRS_RX | V5_SYS | GND UART0 TX -> ELRS RX (GPIO16) 4 R1 ELRS_TX | V5_SYS | GND UART0 RX <- ELRS TX (GPIO17) 5 SDA MAG_SDA | V3V3_SYS | GND I2C1 SDA (GPIO22), 4.7k pull-up on the MCU sheet 6 SCL MAG_SCL | V3V3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"
- note removed: "MECHANICAL: H1-H4 are the four 4.0 mm NPTH grommet holes on the standard 30.5 x 30.5 mm pattern, centred on the board, each with a 5.0 mm copper keepout and an 8.0 mm top-side courtyard for the grommet flange. No pins, no nets. See DESIGN_SPEC "Physical design"."
- note removed: "PWM MAP PWM5 = GPIO20 (row 7, S5) PWM6 = GPIO19 (row 8, S6) PWM7 = GPIO15 (row 9, S7) PWM8 = GPIO5 (row 10, S8) ON THE ESC PAD ROW (J3, POWER 1) PWM1 = GPIO43 PWM2 = GPIO39"
- note removed: "PWM3 = GPIO38 PWM4 = GPIO36"
- note removed: "RAILS ON THE ARRAY: rows 1-4 (GPS, ELRS) and rows 7-10 (servos S5-S8) take V5_SYS; rows 5-6 (magnetometer) and rows 11-14 (the four exposed spares) take V3V3_SYS. Every row has its own GND pin in the J8 column, so a signal return is never more than 2.54 mm away and no row can be mis-plugged into a neighbour's ground. SERVO 5 V NOW COMES FROM V5_SYS, NOT 5V_IN. The old J13 servo row tapped 5V_IN d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"
