File: io_block.kicad_sch (KiCad schematic)
At the start: 10 parts, among them J6 IO array signal column (inner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, J7 IO array power column (5V / 3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, J8 IO array GND column (board ed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

Commit message: Move JLCPCB export to Fabrication Toolkit; drop tools/jlc scripts
- Add fabrication-toolkit-options.json (auto translate + exclude DNP on;
  auto fill, V-cut, alternate outline, all-active-layer plotting off)
- Mark hand-soldered headers and board-only footprints excluded from
  BOM/position files in both schematic and PCB (U24 stays DNP)
- Remove tools/jlc/*, tools/jlc/lcsc_map.csv and power_bom.csv;
  the plugin now produces production/{MARV-V2.zip,bom.csv,positions.csv}
- Ignore generated production/ output; update README and LIBRARIES.md

Verified: 88 top-side placements, 34 LCSC parts, XY identical to prior
export; ERC 0, DRC 0 errors / 0 unconnected / 0 parity issues.

Co-Authored-By: Claude Fable 5.1 <noreply@anthropic.com>
Parts:
- H1, H2, H3, H4, J6, J7, J8: now left out of the parts list
Changed lines of the file:
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@@
 		(body_style 1)
 		(exclude_from_sim no)
-		(in_bom yes)
-		(on_board yes)
-		(in_pos_files yes)
+		(in_bom no)
+		(on_board yes)
+		(in_pos_files no)
 		(dnp no)
 		(property "Reference" "J6"
@@
 		(body_style 1)
 		(exclude_from_sim no)
-		(in_bom yes)
-		(on_board yes)
-		(in_pos_files yes)
+		(in_bom no)
+		(on_board yes)
+		(in_pos_files no)
 		(dnp no)
 		(property "Reference" "J8"
@@
 		(body_style 1)
 		(exclude_from_sim no)
-		(in_bom yes)
-		(on_board yes)
-		(in_pos_files yes)
+		(in_bom no)
+		(on_board yes)
+		(in_pos_files no)
 		(dnp no)
 		(property "Reference" "H3"
@@
 		(body_style 1)
 		(exclude_from_sim no)
-		(in_bom yes)
-		(on_board yes)
-		(in_pos_files yes)
+		(in_bom no)
+		(on_board yes)
+		(in_pos_files no)
 		(dnp no)
 		(property "Reference" "H2"
@@
 		(body_style 1)
 		(exclude_from_sim no)
-		(in_bom yes)
-		(on_board yes)
-		(in_pos_files yes)
+		(in_bom no)
+		(on_board yes)
+		(in_pos_files no)
 		(dnp no)
 		(property "Reference" "H4"
@@
 		(body_style 1)
 		(exclude_from_sim no)
-		(in_bom yes)
-		(on_board yes)
-		(in_pos_files yes)
+		(in_bom no)
+		(on_board yes)
+		(in_pos_files no)
 		(dnp no)
 		(property "Reference" "H1"
@@
 		(body_style 1)
 		(exclude_from_sim no)
-		(in_bom yes)
-		(on_board yes)
-		(in_pos_files yes)
+		(in_bom no)
+		(on_board yes)
+		(in_pos_files no)
 		(dnp no)
 		(property "Reference" "J7"
