File: power_vbat.kicad_sch (KiCad schematic)
At the start: 16 parts, among them J3 ESC pads (CURR TX M4 M3 M2 M1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, U26 AP63205WU-7

Commit message: Power tree: 5 V-in from an external BEC; drop pack buck, TPS2121 mux, TPS62913 stage and USB ESD
Reverses the "pack-powered from the ESC" decision, which was made without
the owner's agreement and inverted the stated requirement (5 V in from a
BEC between the ESC and the FC, so any 2-6S BEC or a 1S boost works
upstream). 140 -> 116 parts; JLC 46 -> 32 LCSC parts, 29 -> 17 Extended.

- J3 ESC row 1x08 -> 1x09: pad 7 5V_IN, pad 8 GND, pad 9 VBAT (sense only,
  feeds the R27/R28/C48 divider on GPIO41; no zone, dropped from Power class)
- USB/5V OR: Q1 AO3401A (gate on USB_VBUS, 100k pull-down) + D1 1N5819WS,
  both JLC Basic. IO-block 5 V rows, C19, C20, C21 move ahead of the FET
  onto 5V_IN; V5_SYS feeds only U7, U12 and the status LED
- 3.3 V system rail: AP63203WU-7 fixed 3.3 V buck on its datasheet
  application circuit (DS41326 Table 2; 4.7 uH FTC404030S reused per sec. 10)
  replaces TPS62913 + FB1 + 0.1 % divider + two-stage filter. JLC Basic has
  no synchronous buck at all, so this one Extended part is accepted
- U12 TPS7A2033 analog LDO kept; EN now tied to V3V3_SYS (PWR_GOOD gone)
- PWR_SRC_ST gone, GPIO37 freed (no-connect); R10 becomes the MCU_RUN pull-up
- U8 USBLC6 (Extended) removed; D+/D- straight to the 27 R series resistors
- ngspice decks that modelled the removed chain retired to
  simulations/superseded/; run_power_checks.py reports RETIRED, not PASS
- DESIGN_SPEC decisions, README, LIBRARIES, PINOUT, BOM, JLC files and
  reports regenerated

Also carries the pre-session working-tree changes (grommet footprint
MountingHole_4.0mm_Grommet -> _Pad_Via, setup_pcb floorplan, JLC tooling).

Verified: ERC 0 violations; check_power_netlist PASS (5V_IN/V5_SYS/VBAT
membership asserted); setup_pcb 0 fit/geometry problems; stitch 150 vias;
DRC 5 silk_edge_clearance warnings only (board unrouted by design);
audit_footprints 116/116; JLC live audit 0 unresolved fitted parts;
generators idempotent modulo UUIDs.

Co-Authored-By: Claude Fable 5.1 <noreply@anthrop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
Parts:
- removed C73: 10u / 50 V X5R 0805 GRM21BR61H106KE43, VIN bulk, Capacitor_SMD:C_0805_2012Metric, symbol Device:C
- removed C74: 100n / 50 V X7R 0402, VIN HF bypass, Capacitor_SMD:C_0402_1005Metric, symbol Device:C
- removed C75: 100n / 50 V X7R 0402, bootstrap, Capacitor_SMD:C_0402_1005Metric, symbol Device:C
- removed C76, C77: 22u / 25 V X5R 0805 GRM21BR61E226ME44, buck COUT, Capacitor_SMD:C_0805_2012Metric, symbol Device:C
- removed C80: 22u / 25 V X5R 0805 GRM21BR61E226ME44, buck COUT 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, Capacitor_SMD:C_0805_2012Metric, symbol Device:C
- removed L3: 4.7u, Isat 6.0 A (30 %), DCR 46 mOhm max (CJIANG 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, MARV_Packages:L_Changjiang_FTC404030S, symbol Device:L
- removed R52: 100k / 1%, EN to VIN, Resistor_SMD:R_0402_1005Metric, symbol Device:R
- removed U26: AP63205WU-7, Package_TO_SOT_SMD:TSOT-23-6, symbol Regulator_Switching:AP63205WU
- added C19: 100u / 6.3 V polymer, ESR <= 40 mOhm (e.g. Panaso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, Capacitor_Tantalum_SMD:CP_EIA-3528-21_Kemet-B, symbol Device:C
- J3: value ESC pads (CURR TX M4 M3 M2 M1 VBAT GND) -> ESC pads (CURR TX M4 M3 M2 M1 5V GND VBAT); footprint MARV_Packages:PadRow_1x08_P2.00mm -> MARV_Packages:PadRow_1x09_P2.00mm; symbol Connector_Generic:Conn_01x08 -> Connector_Generic:Conn_01x09
Connections:
- net 5V_IN: now also J3.7 (Pin_7), C19.1
- net GND: now also C19.2
- net VBAT: now also J3.9 (Pin_9); no longer J3.7 (Pin_7)
Other:
- note added: "5 V in from the external BEC"
- note added: "BOARD INPUTS: REGULATED 5 V FROM AN EXTERNAL BEC on the ESC pad row J3 pin 7 (5V_IN), and USB VBUS ~5 V (J4). There is no on-board pack buck any more (DESIGN_SPEC "Decisions", 2026-09-17): raw pack reaches this board only as the J3 pin 9 SENSE wire VBAT, which drives the R27/R28/C48 divider and nothing else - no load, no bulk, no copper zone. 5V_IN is the servo / GPS / ELRS bus (IO block rows 1-4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"
- note added: "ESC PAD ROW J3 (MicoAir AM32 4-in-1 ESC, FC-connection row), NINE PADS. Pads 1-6 are the ESC silkscreen read left to right; pads 7-9 are this board's power entry, added when the on-board pack buck was removed: 1 CURR - analog current sense from the ESC, 12.75 mV/A, 0-3.3 V -> R53/C78 -> GPIO42 (ADC2) on BOARD 1. 2 TX - KISS ESC telemetry, 3.3 V, 115200 baud, ESC output only -> R54 -> GPIO32 (PIO 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"
- note added: "POWER 1 - ESC PAD ROW J3 (NINE PADS), 5 V INPUT FROM AN EXTERNAL BEC, VBAT SENSE, ANALOG SENSE. Regulated 5 V arrives on J3 pin 7 as 5V_IN; pin 9 brings raw pack VBAT in as a SENSE wire only."
- note removed: "BOARD INPUTS: VBAT 6-25.2 V (2-6S) from the ESC pad row J3, and USB VBUS ~5 V (J4). U26 (AP63205WU) makes 5V_IN from VBAT; 5V_IN is the priority input of the U25 power mux and also the servo 5 V bus."
- note removed: "Buck output bulk (3 x 22 uF)"
- note removed: "ESC PAD ROW J3 (MicoAir AM32 4-in-1 ESC, FC-connection row). Order is the ESC silkscreen read left to right: 1 CURR - analog current sense from the ESC, 12.75 mV/A, 0-3.3 V -> R53/C78 -> GPIO42 (ADC2) on BOARD 1. 2 TX - KISS ESC telemetry, 3.3 V, 115200 baud, ESC output only -> R54 -> GPIO32 (PIO UART RX, GPIOBASE 16 window). 3-6 M4 M3 M2 M1 - 3.3 V DShot/PWM inputs via PIO (GPIOBASE 16 window), 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"
- note removed: "POWER 1 - ESC PAD ROW J3, VBAT INPUT, AP63205 5 V BUCK, ANALOG SENSE. VBAT 6-25.2 V (2-6S) arrives on J3 pin 7; U26 makes 5V_IN from it."
- note removed: "U26 AP63205WU-7 VBAT BUCK (Diodes DS41326 Rev. 2-2). 3.8-32 V in, FIXED 5.0 V out (4.95/5.00/5.05 V, Electrical Characteristics VFB row), 2 A, 1.1 MHz with +/-6% frequency spread spectrum, 4 ms internal soft-start, 22 uA quiescent, TSOT-23-6. VIN abs max 35 V DC / 40 V for 400 ms vs a 25.2 V 6S pack. Component values are Table 3 "Recommended Component Selections for AP63205" and Figure 21 verbati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"
- note removed: "VBAT -> 5V_IN synchronous buck"
- note removed: "VIN bulk at the pin"
- note removed: "case, Irms 3.8 A), is 60 mOhm typ. If height ever has to come out of here, FTC404020S4R7MGCA is the same 4 x 4 land at 2.0 mm tall, but a 2.0 mm core stores less energy: Isat falls to 5.5 A worst case and DCR rises to 58 mOhm max. Ripple at 25.2 V in / 2 A out is 0.78 A pk-pk (Eq.7), peak 2.39 A (Eq.8). DERATING CAVEAT: C73 and C76/C77/C80 are the datasheet nominal values, and ceramic DC-bias der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"
- title: POWER 1 / ESC pad row, VBAT and the 5 V buck -> POWER 1 / ESC pad row, 5 V input and analog sense
