File: power_vbat.kicad_sch (KiCad schematic)
At the start: 8 parts, among them J3 ESC pads (CURR TX M4 M3 M2 M1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

Commit message: update
Parts:
- J3: now in the parts list
Changed lines of the file:
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@@
 		(body_style 1)
 		(exclude_from_sim no)
-		(in_bom no)
+		(in_bom yes)
 		(on_board yes)
-		(in_pos_files no)
+		(in_pos_files yes)
 		(dnp no)
 		(property "Reference" "J3"
