File: usb_debug.kicad_sch (KiCad schematic)
At the start: 11 parts, among them J10 DBG pads (SWCLK SWDIO GND), J4 USB_C_PROGRAM_POWER, U8 USBLC6-2SC6

Commit message: Power tree: 5 V-in from an external BEC; drop pack buck, TPS2121 mux, TPS62913 stage and USB ESD
Reverses the "pack-powered from the ESC" decision, which was made without
the owner's agreement and inverted the stated requirement (5 V in from a
BEC between the ESC and the FC, so any 2-6S BEC or a 1S boost works
upstream). 140 -> 116 parts; JLC 46 -> 32 LCSC parts, 29 -> 17 Extended.

- J3 ESC row 1x08 -> 1x09: pad 7 5V_IN, pad 8 GND, pad 9 VBAT (sense only,
  feeds the R27/R28/C48 divider on GPIO41; no zone, dropped from Power class)
- USB/5V OR: Q1 AO3401A (gate on USB_VBUS, 100k pull-down) + D1 1N5819WS,
  both JLC Basic. IO-block 5 V rows, C19, C20, C21 move ahead of the FET
  onto 5V_IN; V5_SYS feeds only U7, U12 and the status LED
- 3.3 V system rail: AP63203WU-7 fixed 3.3 V buck on its datasheet
  application circuit (DS41326 Table 2; 4.7 uH FTC404030S reused per sec. 10)
  replaces TPS62913 + FB1 + 0.1 % divider + two-stage filter. JLC Basic has
  no synchronous buck at all, so this one Extended part is accepted
- U12 TPS7A2033 analog LDO kept; EN now tied to V3V3_SYS (PWR_GOOD gone)
- PWR_SRC_ST gone, GPIO37 freed (no-connect); R10 becomes the MCU_RUN pull-up
- U8 USBLC6 (Extended) removed; D+/D- straight to the 27 R series resistors
- ngspice decks that modelled the removed chain retired to
  simulations/superseded/; run_power_checks.py reports RETIRED, not PASS
- DESIGN_SPEC decisions, README, LIBRARIES, PINOUT, BOM, JLC files and
  reports regenerated

Also carries the pre-session working-tree changes (grommet footprint
MountingHole_4.0mm_Grommet -> _Pad_Via, setup_pcb floorplan, JLC tooling).

Verified: ERC 0 violations; check_power_netlist PASS (5V_IN/V5_SYS/VBAT
membership asserted); setup_pcb 0 fit/geometry problems; stitch 150 vias;
DRC 5 silk_edge_clearance warnings only (board unrouted by design);
audit_footprints 116/116; JLC live audit 0 unresolved fitted parts;
generators idempotent modulo UUIDs.

Co-Authored-By: Claude Fable 5.1 <noreply@anthrop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
Parts:
- removed U8: USBLC6-2SC6, Package_TO_SOT_SMD:SOT-23-6, symbol Power_Protection:USBLC6-2SC6
Connections:
- net USB_DM_MCU is gone; now on net USB_DM: R23.1
- net USB_DP_MCU is gone; now on net USB_DP: R22.1
Other:
- note added: "BOARD 5 - J4 USB-C 2.0 RECEPTACLE, THE 27 R D+/D- SERIES PAIR, THE VBUS SENSE DIVIDER AND THE J10 SWD LANDING PADS. NO ON-BOARD USB ESD ARRAY - U8 USBLC6 was removed."
- note added: "D+/D- series pair - no ESD array"
- note added: "J10 is a 3-pad SWD landing (SWCLK / SWDIO / GND), not a 10-pin Cortex header: solder pads are kept for the two ports that mate with something fixed - the ESC row J3 and this one (DESIGN_SPEC "Connection philosophy"). The debugger reference 3V3 and the debugger-driven reset line of the old 2x05 header are both gone - power the board from the BEC or USB while debugging, and use SW1 (MCU_RUN to GND)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"
- note added: "USB_VBUS feeds the D1 Schottky and the Q1 gate on POWER 2 directly; no inrush or current limiting on this sheet, and no data ESD array any more - U8 USBLC6-2SC6 was JLC Extended and is removed (DESIGN_SPEC "Decisions"), so D+/D- go straight from J4 into the 27 R series pair R22/R23, as on the madflight FC3v2. The RP2354B USB pins carry their own on-die ESD structures; a board-level array is what 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"
- note removed: "BOARD 5 - J4 USB-C 2.0 RECEPTACLE, U8 USBLC6 DATA ESD, THE 27 R D+/D- SERIES PAIR, THE VBUS SENSE DIVIDER AND THE J10 SWD LANDING PADS."
- note removed: "Data ESD + series pair"
- note removed: "J10 is a 3-pad SWD landing (SWCLK / SWDIO / GND), not a 10-pin Cortex header: solder pads are kept for the two ports that mate with something fixed - the ESC row J3 and this one (DESIGN_SPEC "Connection philosophy"). The debugger reference 3V3 and the debugger-driven reset line of the old 2x05 header are both gone - power the board from VBAT or USB while debugging, and use SW1 (RUN via PWR_GOOD) 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"
- title: BOARD 5 / USB-C, ESD, SWD pads -> BOARD 5 / USB-C, D+/D- series pair, SWD pads
