File: usb_debug.kicad_sch (KiCad schematic)
At the start: 10 parts, among them J10 DBG pads (SWCLK SWDIO GND), J4 USB_C_PROGRAM_POWER

Commit message: updoot
Parts:
- added D21: LED white 0603, USB power, LED_SMD:LED_0603_1608Metric, symbol Device:LED
- added R56: 1k / 1%, USB LED series, Resistor_SMD:R_0402_1005Metric, symbol Device:R
Connections:
- net GND: now also D21.1 (K)
- net USB_VBUS: now also R56.1
- new net USB_LED_A: D21.2 (A), R56.2
Other:
- note added: "D21 / R56 - USB POWER INDICATOR, THE ONLY LED ON THIS BOARD BESIDES THE WS2812C. USB_VBUS -> R56 1 k -> USB_LED_A -> D21 anode, cathode to GND, so it lights whenever a host is plugged in and is dark on BEC-only power - which is exactly the question a bench user asks of this connector, and one the RGB status LED cannot answer because D20 runs off V5_SYS and lights on either source. D21 IS A WHITE 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"
- note added: "USB power LED"
