File: baro.kicad_sch (KiCad schematic)
At the start: 8 parts, among them U22 BMP581 barometer

Commit message: updoot
Parts:
- removed C55: 1u / 10 V X7R 0402, U22 VDD, Capacitor_SMD:C_0402_1005Metric, symbol Device:C
- removed C57: 1u / 10 V X7R 0402, U22 VDDIO, Capacitor_SMD:C_0402_1005Metric, symbol Device:C
- added R57: 4.7k, Resistor_SMD:R_0402_1005Metric, symbol Device:R
- R50: value 10k, BARO_CS pull-up -> 4.7k; LCSC C25744 -> C25900
- TP5: value TP BARO_CS -> TP BARO_SDA
- U22: symbol MARV_Sensors:BMP581 -> MARV_Sensors:BMP581_I2C
Connections:
- net SENS_MISO is gone; now on net GND: U22.5 (ADDR/SDO)
- net V3V3_ANA: now also U22.6 (CSB), R57.1
- removed net BARO_CS: R50.2, TP5.1, U22.6 (CSB)
- net SENS_MOSI renamed BARO_SDA
- net BARO_SDA: now also TP5.1, R57.2
- net SENS_SCK renamed BARO_SCL
- net BARO_SCL: now also R50.2
Other:
- note added: "BOARD 2 - U22 BMP581 BAROMETER: hardware I2C0, powered from V3V3_ANA."
- note added: "I2C pull-ups: 4.7k"
- note added: "U22 BMP581: SCK/SCL = BARO_SCL; SDI/SDA = BARO_SDA; INT = BARO_INT (dedicated GPIO13). CSB is hard-wired to VDDIO / V3V3_ANA for I2C mode. SDO/ADDR is tied to GND: 7-bit address 0x46. R50 and R57 are 4.7k pull-ups to V3V3_ANA on SCL and SDA; no pull-downs. VDDIO and VDD use V3V3_ANA; all VSS pins use GND. C54/C56 remain 100 nF per supply pin."
- note removed: "BOARD 2 - U22 BMP581 BAROMETER on the shared sensor SPI bus, powered from V3V3_ANA."
- note removed: "CSB idle pull-up"
- note removed: "U22 BMP581: CSB = BARO_CS, SDI = SENS_MOSI, SDO = SENS_MISO, SCK = SENS_SCK, INT = BARO_INT. VDDIO and VDD on V3V3_ANA, all three VSS pins to GND."
- moved on the sheet: C56
