File: highg.kicad_sch (KiCad schematic)
At the start: 8 parts, among them U23 ADXL375 high-g accelerometer

Commit message: updoot
Parts:
- removed C58: 100n / 16 V X7R, U23 VS, Capacitor_SMD:C_0402_1005Metric, symbol Device:C
- removed C61: 1u / 10 V X7R 0402, U23 VDD_IO, Capacitor_SMD:C_0402_1005Metric, symbol Device:C
- R51: value 10k, HG_ACC_CS pull-up -> 10k, ADXL_CS pull-up
- TP10: value TP HG_ACC_INT -> TP ADXL_INT1
- TP6: value TP HG_ACC_CS -> TP ADXL_CS
Connections:
- net ADXL_INT2: now reaches U23.9 (INT2)
- net HG_ACC_CS renamed ADXL_CS
- net HG_ACC_INT renamed ADXL_INT1
- net SENS_MISO renamed ADXL_MISO
- net SENS_MOSI renamed ADXL_MOSI
- net SENS_SCK renamed ADXL_SCK
- no-connect marks 2 -> 1
Other:
- note added: "BOARD 2 - U23 ADXL375: dedicated hardware SPI0 (4-wire). Powered from V3V3_ANA."
- note added: "the BMP581 datasheet gives no external-component BOM and asks for no supply capacitor, so 100 nF each is the minimum HF bypass rather than a datasheet value, and the 1 uF C55/C57 that used to sit beside them are gone. U23 ADXL375: CS = ADXL_CS, SDA/SDI = ADXL_MOSI, SDO = ADXL_MISO, SCL/SCLK = ADXL_SCK, INT1 = ADXL_INT1. Per the pin function table, pin 3 (RESERVED) goes to VS and pin 11 (RESERVED)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"
- note removed: "BOARD 2 - U23 ADXL375 HIGH-G ACCELEROMETER on the shared sensor SPI bus, from V3V3_ANA."
- note removed: "U23 ADXL375: CS = HG_ACC_CS, SDA/SDI = SENS_MOSI, SDO = SENS_MISO, SCL/SCLK = SENS_SCK, INT1 = HG_ACC_INT. Per the pin function table, pin 3 (RESERVED) goes to VS and pin 11 (RESERVED) to GND; pin 10 (NC) and the unused INT2 are left open. VS and VDD I/O are both on V3V3_ANA."
- moved on the sheet: C59, C60
