File: imu.kicad_sch (KiCad schematic)
At the start: 12 parts, among them U21 ICM-45686 6-axis IMU

Commit message: updoot
Parts:
- removed C51: 1u / 10 V X7R 0402, U21 VDD, Capacitor_SMD:C_0402_1005Metric, symbol Device:C
- removed C53: 1u / 10 V X7R 0402, U21 VDDIO, Capacitor_SMD:C_0402_1005Metric, symbol Device:C
- R48: value 10k, IMU_CS pull-up -> 10k, ICM_CS pull-up
- TP1: value TP SENS_SCK -> TP ICM_SCK
- TP2: value TP SENS_MOSI -> TP ICM_MOSI
- TP3: value TP SENS_MISO -> TP ICM_MISO
- TP4: value TP IMU_CS -> TP ICM_CS
- TP7: value TP IMU_INT1 -> TP ICM_INT1
- TP8: value TP IMU_INT2 -> TP ICM_INT2
Connections:
- net IMU_CS renamed ICM_CS
- net IMU_INT1 renamed ICM_INT1
- net IMU_INT2 renamed ICM_INT2
- net SENS_MISO renamed ICM_MISO
- net SENS_MOSI renamed ICM_MOSI
- net SENS_SCK renamed ICM_SCK
Other:
- note added: "BOARD 2 - U21 ICM-45686: dedicated hardware SPI1. Powered from V3V3_ANA."
- note added: "Dedicated buses: ADXL375 on hardware SPI0; ICM-45686 on hardware SPI1; BMP581 on hardware I2C0. All sensors use V3V3_ANA. Existing supply decoupling is retained. ICM-45686: C50/C52 are 100 nF X7R on VDD/VDDIO per datasheet Table 11."
- note added: "R48: 10k from ICM_CS to V3V3_ANA; R51: 10k from ADXL_CS to V3V3_ANA. CS pull-ups hold each sensor deselected during reset. No pulls on SPI clock/data. ICM_INT1 and ICM_INT2 each have their own MCU GPIO, independent of all other sensors."
- note added: "Test points: TP1 ICM_SCK, TP2 ICM_MOSI, TP3 ICM_MISO, TP4 ICM_CS; TP5 BARO_SDA, TP6 ADXL_CS; TP7 ICM_INT1, TP8 ICM_INT2, TP9 BARO_INT, TP10 ADXL_INT1. Keep probe stubs short. Routing priority: ICM SPI, ADXL SPI, native SD, then BMP581 I2C. Use a continuous ground reference; avoid switching nodes and long runs beside servo/pyro power."
- note added: "U21 ICM-45686 (TDK InvenSense DS-000577 Rev 1.0, Table 10 "Signal Descriptions" / Figure 4 pin-out, Single Interface SPI mode, Figure 10): AP_CS (pin 12) = ICM_CS, AP_SCLK (13) = ICM_SCK, AP_SDA/AP_SDIO/AP_SDI (14) = ICM_MOSI, AP_SDO/AP_AD0 (1) = ICM_MISO. INT1 (4) = ICM_INT1. INT2/FSYNC/CLKIN (9) = ICM_INT2 - typed bidirectional because FSYNC/CLKIN are host-driven inputs while INT2 is a chip out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"
- note removed: "All three sensors run 4-wire SPI on the shared SENS_SCK / SENS_MOSI / SENS_MISO bus with one chip select each, and are powered from V3V3_ANA (TPS7A20 LDO). Every supply pin on this sheet gets 100 nF + 1 uF: BMP581 and ADXL375 because their own datasheets call for the pair, the ICM-45686 as a deliberate addition - its datasheet BOM (DS-000577 Rev 1.0 Table 11) lists 0.1 uF only."
- note removed: "BOARD 2 - U21 ICM-45686 6-AXIS IMU on the shared sensor SPI bus, powered from V3V3_ANA."
- note removed: "R48, R50, R51: 10k pull-ups to V3V3_ANA on the three SPI chip selects (IMU_CS, BARO_CS, HG_ACC_CS). R49 (the former second IMU chip-select pull-up) is removed along with that net - the ICM-45686 has a single chip select. Same rationale as R35 on FLASH_CS1 (BOARD 3): every sensor is held deselected before the RP2354B drives the pin, so a GPIO left floating through reset, BOOTSEL or a debugger halt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"
- note removed: "TEST POINTS TP1-TP10 (TestPoint:TestPoint_Pad_1.0x1.0mm, 1 x 1 mm bare F.Cu pad, no 3D model by design - tools/audit_footprints.py --no-3d-ok covers ^TestPoint_ along with the pad rows and mounting holes). TP1 SENS_SCK | TP2 SENS_MOSI | TP3 SENS_MISO | TP4 IMU_CS | TP5 BARO_CS | TP6 HG_ACC_CS | TP7 IMU_INT1 | TP8 IMU_INT2 | TP9 BARO_INT | TP10 HG_ACC_INT. Placement: inside the sensor cluster, wit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"
- note removed: "U21 ICM-45686 (TDK InvenSense DS-000577 Rev 1.0, Table 10 "Signal Descriptions" / Figure 4 pin-out, Single Interface SPI mode, Figure 10): AP_CS (pin 12) = IMU_CS, AP_SCLK (13) = SENS_SCK, AP_SDA/AP_SDIO/AP_SDI (14) = SENS_MOSI, AP_SDO/AP_AD0 (1) = SENS_MISO. INT1 (4) = IMU_INT1. INT2/FSYNC/CLKIN (9) = IMU_INT2 - typed bidirectional because FSYNC/CLKIN are host-driven inputs while INT2 is a chip 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"
- moved on the sheet: C52
