File: imu.kicad_sch (KiCad schematic)
At the start: 10 parts, among them U21 ICM-45686 6-axis IMU

Commit message: Normalise silkscreen for JLC, reorder MCU GPIOs, relax DFM guards
- Silk strokes 0.15 mm, silk text 1.0/0.15 mm, no outlines on 0402 R/C and L2,
  compact no-silk test-point footprint (MARV_Packages), edge-connector silk
  trimmed inside the outline, one dangling GND via removed;
  lib_footprint_mismatch set to ignore in the DFM profile and documented.
- MCU pin order: SD bus on GPIO28-33 (top-left corner), ESC row in J3 pad order
  (TELEM GPIO34, PWM4-1 GPIO36-39, CURR ADC1, VBAT ADC2), LED_DATA GPIO43;
  GPIO26/27/35 no-connect. PINOUT.md, DESIGN_SPEC.md and the netlist checker
  follow.
- IO block J7 rows 7-10 moved from 5V_IN to V3V3_SYS (no servo power from FC).
- DFM: courtyard rules relaxed to JLC body-to-body equivalents, no-surcharge via
  presets 0.45/0.20, 0.50/0.25, 0.60/0.30, via-in-pad rule exempts the back-side
  hand-solder rows J3/J10.

Co-Authored-By: Claude Fable 5.1 <noreply@anthropic.com>
Claude-Session: https://claude.ai/code/session_01VST8gLViyNpcDEYyh3itUW
Parts:
- TP1, TP2, TP3, TP4, TP7, TP8: footprint TestPoint:TestPoint_Pad_1.0x1.0mm -> MARV_Packages:TestPoint_Pad_1.0x1.0mm_Compact
Changed lines of the file:
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@@
 			)
 		)
-		(property "Footprint" "TestPoint:TestPoint_Pad_1.0x1.0mm"
+		(property "Footprint" "MARV_Packages:TestPoint_Pad_1.0x1.0mm_Compact"
 			(at 83.82 125.73 0)
 			(hide yes)
@@
 			)
 		)
-		(property "Footprint" "TestPoint:TestPoint_Pad_1.0x1.0mm"
+		(property "Footprint" "MARV_Packages:TestPoint_Pad_1.0x1.0mm_Compact"
 			(at 134.62 125.73 0)
 			(hide yes)
@@
 			)
 		)
-		(property "Footprint" "TestPoint:TestPoint_Pad_1.0x1.0mm"
+		(property "Footprint" "MARV_Packages:TestPoint_Pad_1.0x1.0mm_Compact"
 			(at 160.02 125.73 0)
 			(hide yes)
@@
 			)
 		)
-		(property "Footprint" "TestPoint:TestPoint_Pad_1.0x1.0mm"
+		(property "Footprint" "MARV_Packages:TestPoint_Pad_1.0x1.0mm_Compact"
 			(at 109.22 125.73 0)
 			(hide yes)
@@
 			)
 		)
-		(property "Footprint" "TestPoint:TestPoint_Pad_1.0x1.0mm"
+		(property "Footprint" "MARV_Packages:TestPoint_Pad_1.0x1.0mm_Compact"
 			(at 58.42 125.73 0)
 			(hide yes)
@@
 			)
 		)
-		(property "Footprint" "TestPoint:TestPoint_Pad_1.0x1.0mm"
+		(property "Footprint" "MARV_Packages:TestPoint_Pad_1.0x1.0mm_Compact"
 			(at 33.02 125.73 0)
 			(hide yes)

Commit message: Move JLCPCB export to Fabrication Toolkit; drop tools/jlc scripts
- Add fabrication-toolkit-options.json (auto translate + exclude DNP on;
  auto fill, V-cut, alternate outline, all-active-layer plotting off)
- Mark hand-soldered headers and board-only footprints excluded from
  BOM/position files in both schematic and PCB (U24 stays DNP)
- Remove tools/jlc/*, tools/jlc/lcsc_map.csv and power_bom.csv;
  the plugin now produces production/{MARV-V2.zip,bom.csv,positions.csv}
- Ignore generated production/ output; update README and LIBRARIES.md

Verified: 88 top-side placements, 34 LCSC parts, XY identical to prior
export; ERC 0, DRC 0 errors / 0 unconnected / 0 parity issues.

Co-Authored-By: Claude Fable 5.1 <noreply@anthropic.com>
Parts:
- TP1, TP2, TP3, TP4, TP7, TP8: now left out of the parts list
Changed lines of the file:
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@@
 		(body_style 1)
 		(exclude_from_sim no)
-		(in_bom yes)
-		(on_board yes)
-		(in_pos_files yes)
+		(in_bom no)
+		(on_board yes)
+		(in_pos_files no)
 		(dnp no)
 		(property "Reference" "TP3"
@@
 		(body_style 1)
 		(exclude_from_sim no)
-		(in_bom yes)
-		(on_board yes)
-		(in_pos_files yes)
+		(in_bom no)
+		(on_board yes)
+		(in_pos_files no)
 		(dnp no)
 		(property "Reference" "TP7"
@@
 		(body_style 1)
 		(exclude_from_sim no)
-		(in_bom yes)
-		(on_board yes)
-		(in_pos_files yes)
+		(in_bom no)
+		(on_board yes)
+		(in_pos_files no)
 		(dnp no)
 		(property "Reference" "TP8"
@@
 		(body_style 1)
 		(exclude_from_sim no)
-		(in_bom yes)
-		(on_board yes)
-		(in_pos_files yes)
+		(in_bom no)
+		(on_board yes)
+		(in_pos_files no)
 		(dnp no)
 		(property "Reference" "TP4"
@@
 		(body_style 1)
 		(exclude_from_sim no)
-		(in_bom yes)
-		(on_board yes)
-		(in_pos_files yes)
+		(in_bom no)
+		(on_board yes)
+		(in_pos_files no)
 		(dnp no)
 		(property "Reference" "TP2"
@@
 		(body_style 1)
 		(exclude_from_sim no)
-		(in_bom yes)
-		(on_board yes)
-		(in_pos_files yes)
+		(in_bom no)
+		(on_board yes)
+		(in_pos_files no)
 		(dnp no)
 		(property "Reference" "TP1"
