File: power_3v3.kicad_sch (KiCad schematic)
At the start: 11 parts, among them U12 TPS7A2033PDBVR, U7 AP63203WU-7

Commit message: updoot
Parts:
- removed C9: 100n / 16 V X7R, VIN HF bypass, Capacitor_SMD:C_0402_1005Metric, symbol Device:C
- C26: value 1u / 10 V X7R 0402, LDO output, ESR <=100 mOhm -> 2.2u / 16 V X5R 0603, LDO output (>=1 uF effective, SBVS338H Sec 7.1.1); footprint Capacitor_SMD:C_0402_1005Metric -> Capacitor_SMD:C_0603_1608Metric; LCSC C52923 -> C23630
Other:
- note removed: "rework one. C19, THE 5V_IN BULK, IS 100 uF / 6.3 V POLYMER IN AN EIA-3528-21 (B) CASE. It moved from V5_SYS to 5V_IN with the BEC decision: hold-up belongs on the rail the servo and module rows are on, which is now ahead of the OR-ing FET, and V5_SYS keeps only C8/C9 at the AP63203 input. ESR must stay <= 40 mOhm: Panasonic 6TPE100MAZB or a KEMET T520/T530 B case. 6.3 V on a 5.0 V rail is a 1.26x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"
