File: qspi_expansion.kicad_sch (KiCad schematic)
At the start: 4 parts, among them U24 DNP: W25Q32JVSNIQ, 32 Mbit QS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

Commit message: updoot
Parts:
- removed C63: 1u / 10 V X7R 0402, U24 VCC (fitted; socket is op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, Capacitor_SMD:C_0402_1005Metric, symbol Device:C
- C62: value 100n / 16 V X7R, U24 VCC (fitted; socket is optional) -> 1u / 10 V X7R 0402, U24 VCC (fitted; socket is optional); LCSC C1525 -> C52923
Other:
- note added: "An OPTIONAL QSPI expansion socket on the shared QSPI bus with GPIO0/QMI CS1n as its chip select, and a latched microSD wired for PIO + DMA native 4-bit SD. Both on V3V3_SYS with local bulk, per the rail split in DESIGN_SPEC. U24 IS DNP - NOT FITTED BY DEFAULT AND NOT IN THE BOM; C62, its bypass, IS fitted, and is a 1 uF: the land is built PSRAM-READY, so no cap has to change when the socket is po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"
- note removed: "An OPTIONAL QSPI expansion socket on the shared QSPI bus with GPIO0/QMI CS1n as its chip select, and a latched microSD wired for 4-bit PIO (also SPI-compatible). Both on V3V3_SYS with local bulk, per the rail split in DESIGN_SPEC. U24, C62 AND C63 ARE DNP - NOT FITTED BY DEFAULT AND NOT IN THE BOM. The land is on the BACK of the board (B.Cu) as a user expansion: firmware and logs use the RP2354B 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"
