File: MARV-V2.kicad_pcb (KiCad board)
At the start: 4 copper layers, 50.7 x 45.5 mm, 107 parts, among them J10 DBG pads (SWCLK SWDIO GND), J11 microSD, Molex 47219-2001 loc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, J3 ESC pads (CURR TX M4 M3 M2 M1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, J4 USB_C_PROGRAM_POWER, J6 IO array signal column (inner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, J7 IO array power column (5V / 3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, J8 IO array GND column (board ed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, Q1 AO3401A, SW1 RESET (RUN to GND), SW2 BOOTSEL (via R24), U12 TPS7A2033PDBVR, U20 RP2354B, U21 ICM-45686 6-axis IMU, U22 BMP581 barometer, U23 ADXL375 high-g accelerometer, U24 DNP: W25Q32JVSNIQ, 32 Mbit QS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, U7 AP63203WU-7, Y1 12 MHz TAXM12M4RFBCCT2T, CL 1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

Commit message: DRC 0 err
Parts:
- L20: value 3.3u, 0806 AOTA-B201610S3R3 -> 3.3u, 0806 AOTA-B201610S3R3-101-T
- moved C39 3.09 mm to (97.8, 107.1), turned to 180 degrees
- moved C45 0.74 mm to (97.8, 108.0)
- moved L20 0.46 mm to (98.2, 109.6)
- moved R39 0.15 mm to (87.0, 92.9)
- moved C62 0.15 mm to (103.2, 107.9)
Routing:
- net BARO_INT: track 18.0 -> 22.1 mm
- net GND: track 84.5 -> 88.6 mm, vias 69 -> 71
- net QSPI_SCLK: track 6.69 -> 10.6 mm
- net V3V3_SYS: track 69.0 -> 72.0 mm
- net DVDD: track 30.8 -> 32.4 mm
- net IO_GPIO47: track 28.3 -> 29.7 mm
- net QSPI_SS: track 13.3 -> 14.7 mm
- net ICM_INT2: track 13.6 -> 12.6 mm
- net MAG_SDA: track 18.4 -> 19.3 mm
- net QSPI_SD0: track 10.1 -> 10.9 mm
- net LED_DATA: track 8.63 -> 7.81 mm
- net FLASH_CS1: track 6.92 -> 7.63 mm
- net ADXL_INT2: track 17.7 -> 18.4 mm
- net MAG_SCL: track 19.2 -> 19.9 mm
- net IO_GPIO44: track 26.0 -> 26.6 mm
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