File: MARV-V2.kicad_pcb (KiCad board)
At the start: 4 copper layers, 50.7 x 45.5 mm, 110 parts, among them J10 SWD header 1x03 2.54 mm (SWCL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, J11 microSD, Molex 47219-2001 loc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, J3 ESC pads (CURR TX M4 M3 M2 M1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, J4 USB_C_PROGRAM_POWER, J6 IO array signal column (inner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, J7 IO array power column (5V / 3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, J8 IO array GND column (board ed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, Q1 AO3401A, SW1 RESET (RUN to GND), SW2 BOOTSEL (via R24), U12 TPS7A2033PDBVR, U20 RP2354B, U21 ICM-45686 6-axis IMU, U22 BMP581 barometer, U23 ADXL375 high-g accelerometer, U24 DNP: W25Q32JVSNIQ, 32 Mbit QS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, U7 AP63203WU-7, Y1 12 MHz TAXM12M4RFBCCT2T, CL 1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

Commit message: update
Parts:
- added G3: Info_SensorTable, MARV_Packages:Info_SensorTable, B.Cu at (93.0, 94.5)
- moved R35 4.83 mm to (105.2, 108.0), turned to 135 degrees
- moved C26 0.97 mm to (105.7, 110.5), turned to 45 degrees
- moved C38 0.95 mm to (100.5, 109.0)
Routing:
- net FLASH_CS1: track 7.63 -> 4.00 mm
- net V3V3_ANA: track 86.7 -> 84.5 mm
- net QSPI_SS: track 14.7 -> 13.7 mm
- net V3V3_SYS: track 72.8 -> 72.1 mm
- net USB_DP_RP: track 12.6 -> 12.0 mm
- net GND: track 90.5 -> 90.1 mm, vias 74 -> 75
Other:
- board text added: "BTSL"
- board text added: "DEBUG"
- board text added: "Designed by Luis Martinez"
- board text added: "RST"
