File: MARV-V2.kicad_pcb (KiCad board)
At the start: 4 copper layers, 50.7 x 45.5 mm, 111 parts, among them J10 SWD header 1x03 2.54 mm (SWCL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, J11 microSD, Molex 47219-2001 loc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, J3 ESC pads (CURR TX M4 M3 M2 M1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, J4 USB_C_PROGRAM_POWER, J6 IO array signal column (inner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, J7 IO array power column (5V / 3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, J8 IO array GND column (board ed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, Q1 AO3401A, SW1 RESET (RUN to GND), SW2 BOOTSEL (via R24), U12 TPS7A2033PDBVR, U20 RP2354B, U21 ICM-45686 6-axis IMU, U22 BMP581 barometer, U23 ADXL375 high-g accelerometer, U24 DNP: W25Q32JVSNIQ, 32 Mbit QS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, U7 AP63203WU-7, Y1 12 MHz TAXM12M4RFBCCT2T, CL 1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

Commit message: update
Parts:
- G2: moved to B.Cu
- U24: moved to F.Cu
- moved G2 15.3 mm to (98.5, 108.6), turned to 180 degrees
- moved C26 9.13 mm to (96.8, 112.5), turned to 180 degrees
- moved U12 7.08 mm to (96.0, 115.0)
- moved C25 7.08 mm to (93.4, 114.5)
- moved R56 6.36 mm to (80.4, 120.3), turned to 180 degrees
- moved U24 6.33 mm to (101.8, 116.5), turned to 90 degrees
- moved D21 5.78 mm to (80.8, 121.6), turned to 180 degrees
- moved R22 5.65 mm to (88.3, 112.8)
- moved R4 5.65 mm to (86.1, 112.8)
- moved R23 5.65 mm to (87.2, 112.8)
- moved R5 5.65 mm to (89.4, 112.8)
- moved J4 5.45 mm to (87.5, 119.1)
- moved R24 5.23 mm to (99.2, 121.0), turned to 180 degrees
- moved SW2 4.71 mm to (95.9, 121.0), turned to 180 degrees
- moved G3 3.35 mm to (96.2, 95.5)
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Routing:
- net GND: track 90.1 -> 75.2 mm, vias 75 -> 74
- net QSPI_SD1: track 5.23 -> 19.6 mm, vias 1 -> 0
- net FLASH_CS1: track 4.00 -> 17.0 mm, vias 1 -> 2
- net QSPI_SD2: track 7.13 -> 14.8 mm, vias 1 -> 0
- net QSPI_SS: track 13.7 -> 20.5 mm, vias 2 -> 0
- net V5_SYS: track 33.2 -> 27.1 mm
- net USB_DP_RP: track 12.0 -> 17.5 mm
- net USB_DM_RP: track 12.7 -> 18.2 mm
- net V3V3_SYS: track 72.1 -> 67.4 mm, vias 25 -> 24
- net IO_GPIO46: track 29.5 -> 27.4 mm
- net USB_VBUS: track 40.1 -> 38.1 mm
- net QSPI_SCLK: track 10.6 -> 8.65 mm, vias 1 -> 0
- net QSPI_SD0: track 10.9 -> 9.01 mm, vias 1 -> 0
- net LED_DATA: track 7.81 -> 9.43 mm
- net IO_GPIO47: track 29.7 -> 28.1 mm
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Other:
- board text removed: "FLASH"
- board text removed: "SOIC-8"

Commit message: update
Parts:
- moved C41 0.92 mm to (95.2, 108.2)
- moved R20 0.72 mm to (94.2, 108.7)
Routing:
- net DVDD: track 37.0 -> 20.2 mm, vias 0 -> 2
- net GND: track 75.2 -> 64.6 mm, vias 74 -> 83
- net VREG_LX: track 4.01 -> 0.00 mm
- net V3V3_ANA: track 83.8 -> 86.2 mm
- net BARO_INT: track 22.1 -> 20.8 mm
- net V3V3_SYS: track 67.4 -> 68.3 mm, vias 24 -> 25
- net IO_GPIO44: track 25.9 -> 26.5 mm
- added copper zone on F.Cu, net DVDD
- added copper zone on F.Cu, net VREG_LX
