File: backups/pre-sheet-reorg-2026-09-16/power_periph.kicad_sch (KiCad schematic)
At the start: 6 parts, among them J6 IO array signal column (inner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, J7 IO array power column (5V / 3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, J8 IO array GND column (board ed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

Commit message: Schematic re-organised into 11 per-subsystem pages, drawn as wired blocks
Each subsystem now has its own sheet (RP2354B, USB/debug, ICM-45686, BMP581,
ADXL375, microSD, QSPI expansion, VBAT buck + ESC row, priority mux, 3.3 V
rail, IO block) with the IC's own decoupling, pull-ups, test points and
connectors placed beside it and wired, labels only for nets leaving the
block. Root sheet is an index. tools/build_power.py grows a small layout
engine (wire routing, junctions, decoupling ladders, note flow) with
self-checks for dangling wires and multi-net wire islands; the long design
notes are preserved verbatim as module constants.

Purely presentational: netlist fingerprint (tools/netlist_fingerprint.py,
new) is identical before and after, ERC 0, power checks pass. PCB footprint
paths re-pointed at the new sheet UUIDs by tools/relink_pcb_paths.py (new);
the board diff is path lines only, DRC unconnected count unchanged.
README/DESIGN_SPEC sheet lists updated; pre-change sheets and generator in
backups/pre-sheet-reorg-2026-09-16/.

Also carries the uncommitted work that preceded it: PCB routing, plane
stitching and route-analysis tools (tools/route_*.py, stitch_planes.py),
GPIO remap in PINOUT.md / check_power_netlist.py / setup_pcb.py, and the
grommet mounting-hole footprint update.

Co-Authored-By: Claude Fable 5.1 <noreply@anthropic.com>
Claude-Session: https://claude.ai/code/session_01Y51PayhRcgfdi3hVsfn4qg
Other:
- note added: "IO ARRAY ROW MAP (row n = J6 pin n signal | J7 pin n power | J8 pin n GND) 1 T0 GPS_RX | V5_SYS | GND UART1 TX -> GPS RX (GPIO24) 2 R0 GPS_TX | V5_SYS | GND UART1 RX <- GPS TX (GPIO25) 3 T1 ELRS_RX | V5_SYS | GND UART0 TX -> ELRS RX (GPIO16) 4 R1 ELRS_TX | V5_SYS | GND UART0 RX <- ELRS TX (GPIO17) 5 SDA MAG_SDA | V3V3_SYS | GND I2C1 SDA (GPIO22), 4.7k pull-up on the MCU sheet 6 SCL MAG_SCL | V3V3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"
- note added: "PWM MAP PWM5 = GPIO20 (row 7, S5) PWM6 = GPIO19 (row 8, S6) PWM7 = GPIO15 (row 9, S7) PWM8 = GPIO5 (row 10, S8) ON THE ESC PAD ROW (J3, POWER 1) PWM1 = GPIO43 PWM2 = GPIO39 PWM3 = GPIO38 PWM4 = GPIO36"
- note removed: "IO ARRAY ROW MAP (row n = J6 pin n signal | J7 pin n power | J8 pin n GND) 1 T0 GPS_RX | V5_SYS | GND UART0 TX -> GPS RX (GPIO12) 2 R0 GPS_TX | V5_SYS | GND UART0 RX <- GPS TX (GPIO13) 3 T1 ELRS_RX | V5_SYS | GND UART1 TX -> ELRS RX (GPIO8) 4 R1 ELRS_TX | V5_SYS | GND UART1 RX <- ELRS TX (GPIO9) 5 SDA MAG_SDA | V3V3_SYS | GND I2C1 SDA (GPIO6), 4.7k pull-up on the MCU sheet 6 SCL MAG_SCL | V3V3_SY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"
- note removed: "PWM MAP PWM5 = GPIO10 (row 7, S5) PWM6 = GPIO11 (row 8, S6) PWM7 = GPIO14 (row 9, S7) PWM8 = GPIO15 (row 10, S8) ON THE ESC PAD ROW (J3, POWER 1) PWM1 = GPIO2 PWM2 = GPIO3 PWM3 = GPIO4 PWM4 = GPIO5"
